Commit message: Adjust async modes.

File: kuka_cybertech_support/urdf/kr_cybertech_ros2_control_macro.xacro (robot description, xacro)
@@ -8,7 +8,11 @@
     </xacro:if>
     <!-- ros2 control -->
+    <xacro:property name="scheduling_policy" value="synchronized"/>
+    <xacro:if value="${mode == 'hardware'}">
+      <xacro:property name="scheduling_policy" value="slave"/>
+    </xacro:if>
     <ros2_control name="${name}" type="system" is_async="true" rw_rate="250">
       <properties>
-        <async scheduling_policy="slave" print_warnings="true" thread_priority="30"/>
+        <async scheduling_policy="${scheduling_policy}" print_warnings="true" thread_priority="30"/>
       </properties>
       <hardware>

File: kuka_fortec_support/urdf/kr_fortec_ros2_control_macro.xacro (robot description, xacro)
@@ -8,7 +8,11 @@
     </xacro:if>
     <!-- ros2 control -->
+    <xacro:property name="scheduling_policy" value="synchronized"/>
+    <xacro:if value="${mode == 'hardware'}">
+      <xacro:property name="scheduling_policy" value="slave"/>
+    </xacro:if>
     <ros2_control name="${name}" type="system" is_async="true" rw_rate="250">
       <properties>
-        <async scheduling_policy="slave" print_warnings="true" thread_priority="30"/>
+        <async scheduling_policy="${scheduling_policy}" print_warnings="true" thread_priority="30"/>
       </properties>
       <hardware>

File: kuka_iontec_support/urdf/kr_iontec_ros2_control_macro.xacro (robot description, xacro)
@@ -8,7 +8,11 @@
     </xacro:if>
     <!-- ros2 control -->
+    <xacro:property name="scheduling_policy" value="synchronized"/>
+    <xacro:if value="${mode == 'hardware'}">
+      <xacro:property name="scheduling_policy" value="slave"/>
+    </xacro:if>
     <ros2_control name="${name}" type="system" is_async="true" rw_rate="250">
       <properties>
-        <async scheduling_policy="slave" print_warnings="true" thread_priority="30"/>
+        <async scheduling_policy="${scheduling_policy}" print_warnings="true" thread_priority="30"/>
       </properties>
       <hardware>

File: kuka_lbr_iisy_support/urdf/lbr_iisy_ros2_control_macro.xacro (robot description, xacro)
@@ -8,7 +8,11 @@
     </xacro:if>
     <!-- ros2 control -->
+    <xacro:property name="scheduling_policy" value="synchronized"/>
+    <xacro:if value="${mode == 'hardware'}">
+      <xacro:property name="scheduling_policy" value="slave"/>
+    </xacro:if>
     <ros2_control name="${name}" type="system" is_async="true" rw_rate="250">
       <properties>
-        <async scheduling_policy="slave" print_warnings="true" thread_priority="30"/>
+        <async scheduling_policy="${scheduling_policy}" print_warnings="true" thread_priority="30"/>
       </properties>
       <hardware>

File: kuka_lbr_iiwa_support/urdf/lbr_iiwa_ros2_control_macro.xacro (robot description, xacro)
@@ -8,9 +8,12 @@
     </xacro:if>
     <!-- ros2 control -->
-    <ros2_control name="${name}" type="system" is_async="true" rw_rate="250">
+    <xacro:property name="scheduling_policy" value="synchronized"/>
+    <xacro:if value="${mode == 'hardware'}">
+      <xacro:property name="scheduling_policy" value="slave"/>
+    </xacro:if>
+    <ros2_control name="${name}" type="system" is_async="true" rw_rate="1000">
       <properties>
-        <async scheduling_policy="slave" print_warnings="true" thread_priority="30"/>
+        <async scheduling_policy="${scheduling_policy}" print_warnings="true" thread_priority="30"/>
       </properties>
-      <hardware>
         <xacro:if value="${mode == 'mock'}">
           <plugin>kuka_mock_hardware_interface::KukaMockHardwareInterface</plugin>

File: kuka_quantec_support/urdf/kr_quantec_ros2_control_macro.xacro (robot description, xacro)
@@ -8,7 +8,11 @@
     </xacro:if>
     <!-- ros2 control -->
+    <xacro:property name="scheduling_policy" value="synchronized"/>
+    <xacro:if value="${mode == 'hardware'}">
+      <xacro:property name="scheduling_policy" value="slave"/>
+    </xacro:if>
     <ros2_control name="${name}" type="system" is_async="true" rw_rate="250">
       <properties>
-        <async scheduling_policy="slave" print_warnings="true" thread_priority="30"/>
+        <async scheduling_policy="${scheduling_policy}" print_warnings="true" thread_priority="30"/>
       </properties>
       <hardware>
