Commit message: Adjust initial positions and joint limits

File: kuka_quantec_support/urdf/kr210_r3100_2_macro.xacro (robot description, xacro)
@@ -20,4 +20,7 @@
         </geometry>
         <origin rpy="-0.0 0.0 -0.0" xyz="0.0 0.0 0.0"/>
+        <material name="custom_blue">
+          <color rgba="0.0 0.6235 0.8902 1.0"/>
+        </material>
       </visual>
     </link>
@@ -39,4 +42,7 @@
         </geometry>
         <origin rpy="-0.0 0.0 -0.0" xyz="0.0 0.0 0.0"/>
+        <material name="custom_blue">
+          <color rgba="0.0 0.6235 0.8902 1.0"/>
+        </material>
       </visual>
     </link>
@@ -58,4 +64,7 @@
         </geometry>
         <origin rpy="-0.0 0.0 -0.0" xyz="0.0 0.0 0.0"/>
+        <material name="custom_blue">
+          <color rgba="0.0 0.6235 0.8902 1.0"/>
+        </material>
       </visual>
     </link>
@@ -77,4 +86,7 @@
         </geometry>
         <origin rpy="-0.0 0.0 -0.0" xyz="0.0 0.0 0.0"/>
+        <material name="custom_blue">
+          <color rgba="0.0 0.6235 0.8902 1.0"/>
+        </material>
       </visual>
     </link>
@@ -96,4 +108,7 @@
         </geometry>
         <origin rpy="-0.0 0.0 -0.0" xyz="0.0 0.0 0.0"/>
+        <material name="custom_blue">
+          <color rgba="0.0 0.6235 0.8902 1.0"/>
+        </material>
       </visual>
     </link>
@@ -115,4 +130,7 @@
         </geometry>
         <origin rpy="-0.0 0.0 -0.0" xyz="0.0 0.0 0.0"/>
+        <material name="custom_blue">
+          <color rgba="0.0 0.6235 0.8902 1.0"/>
+        </material>
       </visual>
     </link>
@@ -134,4 +152,7 @@
         </geometry>
         <origin rpy="-0.0 0.0 -0.0" xyz="0.0 0.0 0.0"/>
+        <material name="custom_blue">
+          <color rgba="0.0 0.6235 0.8902 1.0"/>
+        </material>
       </visual>
     </link>

File: kuka_quantec_support/urdf/kr300_r2700_2_macro.xacro (robot description, xacro)
@@ -11,7 +11,7 @@
       </collision>
       <inertial>
-        <inertia ixx="12.830880390826948" ixy="0.0" ixz="0.0" iyy="9.01196989503174" iyz="0.0" izz="14.295886015581125"/>
+        <inertia ixx="0.0" ixy="0.0" ixz="0.0" iyy="0.0" iyz="0.0" izz="0.0"/>
         <mass value="2.2596E2"/>
-        <origin rpy="-0.050860131411839545 -0.0019883389878402684 1.523148744399526" xyz="-0.05948933351035582 0.002155950610727567 0.20325069304301646"/>
+        <origin rpy="0.0 -0.0 0.0" xyz="0.0 0.0 0.0"/>
       </inertial>
       <visual>
@@ -31,7 +31,7 @@
       </collision>
       <inertial>
-        <inertia ixx="31.78631557136323" ixy="0.0" ixz="0.0" iyy="13.331031863287903" iyz="0.0" izz="34.180672314725456"/>
+        <inertia ixx="31.7863155713632" ixy="0.0" ixz="0.0" iyy="13.3310318632879" iyz="0.0" izz="34.1806723147255"/>
         <mass value="3.6737E2"/>
-        <origin rpy="-0.35119744183070917 -1.2748494702775002 -1.4514723788195054" xyz="0.02826300460026676 0.011134569507580913 -0.23533673952690748"/>
+        <origin rpy="-0.3511974418307098 -1.2748494702775013 -1.451472378819504" xyz="0.0282630046002668 0.011134569507580901 -0.235336739526907"/>
       </inertial>
       <visual>
@@ -50,7 +50,7 @@
       </collision>
       <inertial>
-        <inertia ixx="57.79570981129111" ixy="0.0" ixz="0.0" iyy="5.63272995683346" iyz="0.0" izz="58.55984559100601"/>
+        <inertia ixx="57.7957098112911" ixy="0.0" ixz="0.0" iyy="5.63272995683346" iyz="0.0" izz="58.559845591006"/>
         <mass value="2.3206E2"/>
-        <origin rpy="-2.820395530490075 -1.2181144847004781 1.2776348095029497" xyz="0.4868709816426786 -0.0019029561320348183 -0.11763677497199002"/>
+        <origin rpy="-2.820395530490072 -1.2181144847004783 1.2776348095029488" xyz="0.486870981642679 -0.00190295613203482 -0.11763677497199"/>
       </inertial>
       <visual>
@@ -69,7 +69,7 @@
       </collision>
       <inertial>
-        <inertia ixx="3.511665641677197" ixy="0.0" ixz="0.0" iyy="21.236938206229333" iyz="0.0" izz="22.25683741872681"/>
+        <inertia ixx="3.5116656416772" ixy="0.0" ixz="0.0" iyy="21.2369382062293" iyz="0.0" izz="22.2568374187268"/>
         <mass value="1.9153E2"/>
-        <origin rpy="2.1669667459514144 -0.06384171041203492 -0.054172455510610194" xyz="0.17268469691432153 -0.0754866078421135 0.13713156998903567"/>
+        <origin rpy="2.1669667459514192 -0.06384171041203483 -0.05417245551061014" xyz="0.172684696914322 -0.0754866078421135 0.137131569989036"/>
       </inertial>
       <visual>
@@ -88,7 +88,7 @@
       </collision>
       <inertial>
-        <inertia ixx="0.20114801831278567" ixy="0.0" ixz="0.0" iyy="1.6156024516095273" iyz="0.0" izz="1.6404174473993869"/>
+        <inertia ixx="0.201148018312786" ixy="0.0" ixz="0.0" iyy="1.61560245160953" iyz="0.0" izz="1.64041744739939"/>
         <mass value="4.7942845677E1"/>
-        <origin rpy="1.5709922511064425 -1.391282030791283 -1.5710550346492322" xyz="-8.827699851665032E-6 0.030038038468557137 -0.22035014882022413"/>
+        <origin rpy="1.570992251106443 -1.3912820307912874 -1.5710550346492322" xyz="-8.82769985166503E-6 0.030038038468557102 -0.22035014882022402"/>
       </inertial>
       <visual>
@@ -107,7 +107,7 @@
       </collision>
       <inertial>
-        <inertia ixx="0.3430603374426301" ixy="0.0" ixz="0.0" iyy="0.19689279813434987" iyz="0.0" izz="0.3479764098342267"/>
+        <inertia ixx="0.34306033744263" ixy="0.0" ixz="0.0" iyy="0.19689279813435" iyz="0.0" izz="0.347976409834227"/>
         <mass value="2.3687644624E1"/>
-        <origin rpy="1.6224506086845296 -0.931996732036955 -0.06488528019057813" xyz="0.062409087507206966 2.1098685344562437E-4 -0.06405788459182832"/>
+        <origin rpy="1.6224506086845345 -0.9319967320369543 -0.06488528019058366" xyz="0.062409087507207 2.1098685344562402E-4 -0.0640578845918283"/>
       </inertial>
       <visual>
@@ -126,7 +126,7 @@
       </collision>
       <inertial>
-        <inertia ixx="0.03694112716090631" ixy="0.0" ixz="0.0" iyy="0.03695315329552196" iyz="0.0" izz="0.0482510013261814"/>
+        <inertia ixx="0.0369411271609063" ixy="0.0" ixz="0.0" iyy="0.0369531532955219" iyz="0.0" izz="0.0482510013261814"/>
         <mass value="1.2245718539E1"/>
-        <origin rpy="1.0758644105172148E-4 -9.81246446146609E-5 -0.03310542818452318" xyz="4.595822618513483E-6 -5.5908945912619675E-6 -0.02543618981825055"/>
+        <origin rpy="1.0758644105165322E-4 -9.812464461473523E-5 -0.03310542818383201" xyz="4.5958226185134805E-6 -5.59089459126197E-6 -0.0254361898182505"/>
       </inertial>
       <visual>
@@ -145,5 +145,5 @@
       <axis xyz="0.0 0.0 1.0"/>
       <child link="${prefix}link_1"/>
-      <limit effort="7.29E3" lower="-3.2288591125E0" upper="3.2288591125E0" velocity="1.8325957145940461E0"/>
+      <limit effort="7.29E3" lower="-3.2288591125E0" upper="3.2288591125E0" velocity="1.83259571459405E0"/>
       <origin rpy="3.141592653589793 -0.0 0.0" xyz="0.0 0.0 0.30560000000000004"/>
       <parent link="${prefix}base_link"/>
@@ -152,5 +152,5 @@
       <axis xyz="0.0 0.0 1.0"/>
       <child link="${prefix}link_2"/>
-      <limit effort="9.60003E3" lower="-2.44346095E0" upper="-8.72664625E-2" velocity="1.7627825445142729E0"/>
+      <limit effort="9.60003E3" lower="-2.44346095E0" upper="-8.72664625E-2" velocity="1.76278254451427E0"/>
       <origin rpy="1.5707963267948966 -0.0 0.0" xyz="0.33 0.07200000000000001 -0.3394"/>
       <parent link="${prefix}link_1"/>
@@ -159,5 +159,5 @@
       <axis xyz="0.0 0.0 1.0"/>
       <child link="${prefix}link_3"/>
-      <limit effort="7.08714342281144E3" lower="-2.0943951E0" upper="2.93215314E0" velocity="1.8675022996339325E0"/>
+      <limit effort="7.08714342281144E3" lower="-2.0943951E0" upper="2.93215314E0" velocity="1.86750229963393E0"/>
       <origin rpy="0.0 -0.0 0.0" xyz="1.1500000000000001 0.0 -0.10300000000000001"/>
       <parent link="${prefix}link_2"/>
@@ -166,5 +166,5 @@
       <axis xyz="0.0 0.0 1.0"/>
       <child link="${prefix}link_4"/>
-      <limit effort="2.25887888718356E3" lower="-6.108652375E0" upper="6.108652375E0" velocity="2.4434609527920612E0"/>
+      <limit effort="2.25887888718356E3" lower="-6.108652375E0" upper="6.108652375E0" velocity="2.44346095279206E0"/>
       <origin rpy="1.5707963267948966 -0.0 -1.5707963267948966" xyz="0.8280000000000001 -0.115 0.17500000000000002"/>
       <parent link="${prefix}link_3"/>
@@ -173,5 +173,5 @@
       <axis xyz="0.0 0.0 1.0"/>
       <child link="${prefix}link_5"/>
-      <limit effort="2.26120660090655E3" lower="-2.13802833125E0" upper="2.13802833125E0" velocity="1.9722220547535925E0"/>
+      <limit effort="2.26120660090655E3" lower="-2.13802833125E0" upper="2.13802833125E0" velocity="1.97222205475359E0"/>
       <origin rpy="0.0 1.5707963267948966 1.5707963267948966" xyz="0.0 0.1065 -0.392"/>
       <parent link="${prefix}link_4"/>
@@ -180,5 +180,5 @@
       <axis xyz="0.0 0.0 1.0"/>
       <child link="${prefix}link_6"/>
-      <limit effort="1.46107811041986E3" lower="-6.108652375E0" upper="6.108652375E0" velocity="3.1415926535897931E0"/>
+      <limit effort="1.46107811041986E3" lower="-6.108652375E0" upper="6.108652375E0" velocity="3.14159265358979E0"/>
       <origin rpy="1.5707963267948966 -0.0 -1.5707963267948966" xyz="0.1695 0.0 -0.1065"/>
       <parent link="${prefix}link_5"/>

File: kuka_quantec_support/urdf/kr_quantec_ros2_control_macro.xacro (robot description, xacro)
@@ -79,5 +79,5 @@
         <command_interface name="position"/>
         <state_interface name="position">
-          <param name="initial_value">0.0</param>
+          <param name="initial_value">1.5708</param>
         </state_interface>
       </joint>
