Commit message: Add orange color to the kr210_r3100_2 model

File: kuka_quantec_support/urdf/kr210_r3100_2_macro.xacro (robot description, xacro)
@@ -20,4 +20,5 @@
         </geometry>
         <origin rpy="-0.0 0.0 -0.0" xyz="0.0 0.0 0.0"/>
+        <material name="kuka_orange"><color rgba="1.0 0.48 0.0 1.0"/></material>
       </visual>
     </link>
@@ -39,4 +40,5 @@
         </geometry>
         <origin rpy="-0.0 0.0 -0.0" xyz="0.0 0.0 0.0"/>
+        <material name="kuka_orange"><color rgba="1.0 0.48 0.0 1.0"/></material>
       </visual>
     </link>
@@ -58,4 +60,5 @@
         </geometry>
         <origin rpy="-0.0 0.0 -0.0" xyz="0.0 0.0 0.0"/>
+        <material name="kuka_orange"><color rgba="1.0 0.48 0.0 1.0"/></material>
       </visual>
     </link>
@@ -77,4 +80,5 @@
         </geometry>
         <origin rpy="-0.0 0.0 -0.0" xyz="0.0 0.0 0.0"/>
+        <material name="kuka_orange"><color rgba="1.0 0.48 0.0 1.0"/></material>
       </visual>
     </link>
@@ -96,4 +100,5 @@
         </geometry>
         <origin rpy="-0.0 0.0 -0.0" xyz="0.0 0.0 0.0"/>
+        <material name="kuka_orange"><color rgba="1.0 0.48 0.0 1.0"/></material>
       </visual>
     </link>
@@ -115,4 +120,5 @@
         </geometry>
         <origin rpy="-0.0 0.0 -0.0" xyz="0.0 0.0 0.0"/>
+        <material name="kuka_orange"><color rgba="1.0 0.48 0.0 1.0"/></material>
       </visual>
     </link>
@@ -134,4 +140,5 @@
         </geometry>
         <origin rpy="-0.0 0.0 -0.0" xyz="0.0 0.0 0.0"/>
+        <material name="kuka_orange"><color rgba="1.0 0.48 0.0 1.0"/></material>
       </visual>
     </link>

Commit message: Fix arm colors
Use predefined materials in kuka_ressources

File: kuka_quantec_support/urdf/kr210_r3100_2_macro.xacro (robot description, xacro)
@@ -1,4 +1,5 @@
 <?xml version="1.0"?>
 <robot xmlns:xacro="http://wiki.ros.org/xacro">
+  <xacro:include filename="$(find kuka_resources)/urdf/common_materials.xacro"/>
   <xacro:macro name="kuka_kr210_r3100_2_robot" params="prefix package_name">
     <!-- links - main serial chain -->
@@ -20,5 +21,5 @@
         </geometry>
         <origin rpy="-0.0 0.0 -0.0" xyz="0.0 0.0 0.0"/>
-        <material name="kuka_orange"><color rgba="1.0 0.48 0.0 1.0"/></material>
+        <xacro:material_kuka_black/>
       </visual>
     </link>
@@ -40,5 +41,5 @@
         </geometry>
         <origin rpy="-0.0 0.0 -0.0" xyz="0.0 0.0 0.0"/>
-        <material name="kuka_orange"><color rgba="1.0 0.48 0.0 1.0"/></material>
+        <xacro:material_kuka_orange/>
       </visual>
     </link>
@@ -60,5 +61,5 @@
         </geometry>
         <origin rpy="-0.0 0.0 -0.0" xyz="0.0 0.0 0.0"/>
-        <material name="kuka_orange"><color rgba="1.0 0.48 0.0 1.0"/></material>
+        <xacro:material_kuka_orange/>
       </visual>
     </link>
@@ -80,5 +81,5 @@
         </geometry>
         <origin rpy="-0.0 0.0 -0.0" xyz="0.0 0.0 0.0"/>
-        <material name="kuka_orange"><color rgba="1.0 0.48 0.0 1.0"/></material>
+        <xacro:material_kuka_orange/>
       </visual>
     </link>
@@ -100,5 +101,5 @@
         </geometry>
         <origin rpy="-0.0 0.0 -0.0" xyz="0.0 0.0 0.0"/>
-        <material name="kuka_orange"><color rgba="1.0 0.48 0.0 1.0"/></material>
+        <xacro:material_kuka_orange/>
       </visual>
     </link>
@@ -120,5 +121,5 @@
         </geometry>
         <origin rpy="-0.0 0.0 -0.0" xyz="0.0 0.0 0.0"/>
-        <material name="kuka_orange"><color rgba="1.0 0.48 0.0 1.0"/></material>
+        <xacro:material_kuka_orange/>
       </visual>
     </link>
@@ -140,5 +141,5 @@
         </geometry>
         <origin rpy="-0.0 0.0 -0.0" xyz="0.0 0.0 0.0"/>
-        <material name="kuka_orange"><color rgba="1.0 0.48 0.0 1.0"/></material>
+        <xacro:material_kuka_orange/>
       </visual>
     </link>
