Commit message: Added world - base_link joint

File: kuka_kr10_description/urdf/kr10r1100sixx.xacro (robot description, xacro)
@@ -6,6 +6,15 @@
     <xacro:arg name="eki_robot_port" default="54600"/>
     <xacro:arg name="use_fake_hardware" default="true"/>
-    <xacro:kuka_kr10r1100sixx prefix="" initial_positions_file="$(arg initial_positions_file)"
+    <xacro:arg name="prefix" default=""/>
+    <xacro:kuka_kr10r1100sixx prefix="$(arg prefix)" initial_positions_file="$(arg initial_positions_file)"
                               robot_ip="$(arg robot_ip)" eki_robot_port="$(arg eki_robot_port)"
                               use_fake_hardware="$(arg use_fake_hardware)"/>
+    <!-- world link -->
+    <link name="world"/>
+    <!-- default world - base_link joint -->
+    <joint name="$(arg prefix)world-base_link" type="fixed">
+        <parent link="world"/>
+        <child link="$(arg prefix)base_link"/>
+        <origin xyz="0 0 0" rpy="0 0 0"/>
+    </joint>
 </robot>

File: kuka_kr10_description/urdf/kr10r900_2.xacro (robot description, xacro)
@@ -6,6 +6,15 @@
     <xacro:arg name="eki_robot_port" default="54600"/>
     <xacro:arg name="use_fake_hardware" default="true"/>
-    <xacro:kuka_kr10r900_2 prefix="" initial_positions_file="$(arg initial_positions_file)"
+    <xacro:arg name="prefix" default=""/>
+    <xacro:kuka_kr10r900_2 prefix="$(arg prefix)" initial_positions_file="$(arg initial_positions_file)"
                            robot_ip="$(arg robot_ip)" eki_robot_port="$(arg eki_robot_port)"
                            use_fake_hardware="$(arg use_fake_hardware)"/>
+    <!-- world link -->
+    <link name="world"/>
+    <!-- default world - base_link joint -->
+    <joint name="$(arg prefix)world-base_link" type="fixed">
+        <parent link="world"/>
+        <child link="$(arg prefix)base_link"/>
+        <origin xyz="0 0 0" rpy="0 0 0"/>
+    </joint>
 </robot>

Commit message: Removed world base_link joint
Already defined in AIP cell xacro

File: kuka_kr10_description/urdf/kr10r1100sixx.xacro (robot description, xacro)
@@ -10,11 +10,3 @@
                               robot_ip="$(arg robot_ip)" eki_robot_port="$(arg eki_robot_port)"
                               use_fake_hardware="$(arg use_fake_hardware)"/>
-    <!-- world link -->
-    <link name="world"/>
-    <!-- default world - base_link joint -->
-    <joint name="$(arg prefix)world-base_link" type="fixed">
-        <parent link="world"/>
-        <child link="$(arg prefix)base_link"/>
-        <origin xyz="0 0 0" rpy="0 0 0"/>
-    </joint>
 </robot>

File: kuka_kr10_description/urdf/kr10r900_2.xacro (robot description, xacro)
@@ -10,11 +10,3 @@
                            robot_ip="$(arg robot_ip)" eki_robot_port="$(arg eki_robot_port)"
                            use_fake_hardware="$(arg use_fake_hardware)"/>
-    <!-- world link -->
-    <link name="world"/>
-    <!-- default world - base_link joint -->
-    <joint name="$(arg prefix)world-base_link" type="fixed">
-        <parent link="world"/>
-        <child link="$(arg prefix)base_link"/>
-        <origin xyz="0 0 0" rpy="0 0 0"/>
-    </joint>
 </robot>

Commit message: Replaced eki hwi with the drivers found in kuka_drivers

File: kuka_kr10_description/urdf/kr10r1100sixx.xacro (robot description, xacro)
@@ -3,10 +3,26 @@
     <xacro:include filename="$(find kuka_kr10_description)/urdf/kr10r1100sixx_macro.xacro"/>
     <xacro:arg name="initial_positions_file" default="$(find kuka_kr10_description)/config/initial_positions.yaml"/>
-    <xacro:arg name="robot_ip" default="10.181.116.41"/>
-    <xacro:arg name="eki_robot_port" default="54600"/>
-    <xacro:arg name="use_fake_hardware" default="true"/>
     <xacro:arg name="prefix" default=""/>
-    <xacro:kuka_kr10r1100sixx prefix="$(arg prefix)" initial_positions_file="$(arg initial_positions_file)"
-                              robot_ip="$(arg robot_ip)" eki_robot_port="$(arg eki_robot_port)"
-                              use_fake_hardware="$(arg use_fake_hardware)"/>
+    <xacro:arg name="driver_version" default="eki_rsi"/>
+    <xacro:arg name="controller_ip" default="10.181.116.41"/>
+    <xacro:arg name="client_ip" default=""/>
+    <xacro:arg name="client_port" default="59152"/>
+    <xacro:arg name="mxa_client_port" default="44444"/>
+    <xacro:arg name="mode" default="mock"/>
+    <xacro:arg name="use_gpio" default="false"/>
+    <xacro:arg name="roundtrip_time" default="0"/>
+    <xacro:arg name="verify_robot_model" default="False"/>
+    <xacro:kuka_kr10r1100sixx prefix="$(arg prefix)"
+                              initial_positions_file="$(arg initial_positions_file)"
+                              driver_version="$(arg driver_version)"
+                              controller_ip="$(arg controller_ip)"
+                              client_ip="$(arg client_ip)"
+                              client_port="$(arg client_port)"
+                              mxa_client_port="$(arg mxa_client_port)"
+                              mode="$(arg mode)"
+                              use_gpio="$(arg use_gpio)"
+                              roundtrip_time="$(arg roundtrip_time)"
+                              verify_robot_model="$(arg verify_robot_model)">
+        <ext_axes_ros2_control_joints/>
+    </xacro:kuka_kr10r1100sixx>
 </robot>

File: kuka_kr10_description/urdf/kr10r1100sixx_macro.xacro (robot description, xacro)
@@ -4,5 +4,5 @@
     <xacro:include filename="$(find kuka_resources)/urdf/common_materials.xacro"/>
     <xacro:include filename="$(find kuka_kr10_description)/urdf/kuka.ros2_control.xacro"/>
-    <xacro:macro name="kuka_kr10r1100sixx" params="prefix initial_positions_file robot_ip eki_robot_port use_fake_hardware">
+    <xacro:macro name="kuka_kr10r1100sixx" params="prefix initial_positions_file driver_version client_ip client_port mxa_client_port controller_ip mode use_gpio roundtrip_time verify_robot_model **ext_axes_ros2_control_joints">
         <link name="${prefix}base_link">
             <visual>
@@ -175,6 +175,17 @@
         <xacro:kuka_ros2_control name="kuka_control" robot_prefix="${prefix}"
                                  initial_positions_file="${initial_positions_file}"
-                                 robot_ip="${robot_ip}" eki_robot_port="${eki_robot_port}"
-                                 use_fake_hardware="${use_fake_hardware}"/>
+                                 driver_version="${driver_version}"
+                                 client_ip="${client_ip}"
+                                 client_port="${client_port}"
+                                 mxa_client_port="${mxa_client_port}"
+                                 controller_ip="${controller_ip}"
+                                 mode="${mode}"
+                                 use_gpio="${use_gpio}"
+                                 roundtrip_time="${roundtrip_time}"
+                                 verify_robot_model="${verify_robot_model}">
+            <ext_axes_ros2_control_joints>
+                <xacro:insert_block name="ext_axes_ros2_control_joints"/>
+            </ext_axes_ros2_control_joints>
+        </xacro:kuka_ros2_control>
     </xacro:macro>
 </robot>

File: kuka_kr10_description/urdf/kr10r900_2.xacro (robot description, xacro)
@@ -3,10 +3,26 @@
     <xacro:include filename="$(find kuka_kr10_description)/urdf/kr10r900_2_macro.xacro"/>
     <xacro:arg name="initial_positions_file" default="$(find kuka_kr10_description)/config/initial_positions.yaml"/>
-    <xacro:arg name="robot_ip" default="10.181.116.41"/>
-    <xacro:arg name="eki_robot_port" default="54600"/>
-    <xacro:arg name="use_fake_hardware" default="true"/>
     <xacro:arg name="prefix" default=""/>
-    <xacro:kuka_kr10r900_2 prefix="$(arg prefix)" initial_positions_file="$(arg initial_positions_file)"
-                           robot_ip="$(arg robot_ip)" eki_robot_port="$(arg eki_robot_port)"
-                           use_fake_hardware="$(arg use_fake_hardware)"/>
+    <xacro:arg name="driver_version" default="eki_rsi"/>
+    <xacro:arg name="controller_ip" default="10.181.116.41"/>
+    <xacro:arg name="client_ip" default=""/>
+    <xacro:arg name="client_port" default="59152"/>
+    <xacro:arg name="mxa_client_port" default="44444"/>
+    <xacro:arg name="mode" default="mock"/>
+    <xacro:arg name="use_gpio" default="false"/>
+    <xacro:arg name="roundtrip_time" default="0"/>
+    <xacro:arg name="verify_robot_model" default="False"/>
+    <xacro:kuka_kr10r900_2 prefix="$(arg prefix)"
+                           initial_positions_file="$(arg initial_positions_file)"
+                           driver_version="$(arg driver_version)"
+                           controller_ip="$(arg controller_ip)"
+                           client_ip="$(arg client_ip)"
+                           client_port="$(arg client_port)"
+                           mxa_client_port="$(arg mxa_client_port)"
+                           mode="$(arg mode)"
+                           use_gpio="$(arg use_gpio)"
+                           roundtrip_time="$(arg roundtrip_time)"
+                           verify_robot_model="$(arg verify_robot_model)">
+        <ext_axes_ros2_control_joints/>
+    </xacro:kuka_kr10r900_2>
 </robot>

File: kuka_kr10_description/urdf/kr10r900_2_macro.xacro (robot description, xacro)
@@ -3,5 +3,5 @@
     <xacro:include filename="$(find kuka_resources)/urdf/common_materials.xacro"/>
     <xacro:include filename="$(find kuka_kr10_description)/urdf/kuka.ros2_control.xacro"/>
-    <xacro:macro name="kuka_kr10r900_2" params="prefix initial_positions_file robot_ip eki_robot_port use_fake_hardware">
+    <xacro:macro name="kuka_kr10r900_2" params="prefix initial_positions_file driver_version client_ip client_port mxa_client_port controller_ip mode use_gpio roundtrip_time verify_robot_model **ext_axes_ros2_control_joints">
         <link name="${prefix}base_link">
             <visual>
@@ -175,6 +175,17 @@
         <xacro:kuka_ros2_control name="kuka_control" robot_prefix="${prefix}"
                                  initial_positions_file="${initial_positions_file}"
-                                 robot_ip="${robot_ip}" eki_robot_port="${eki_robot_port}"
-                                 use_fake_hardware="${use_fake_hardware}"/>
+                                 driver_version="${driver_version}"
+                                 client_ip="${client_ip}"
+                                 client_port="${client_port}"
+                                 mxa_client_port="${mxa_client_port}"
+                                 controller_ip="${controller_ip}"
+                                 mode="${mode}"
+                                 use_gpio="${use_gpio}"
+                                 roundtrip_time="${roundtrip_time}"
+                                 verify_robot_model="${verify_robot_model}">
+            <ext_axes_ros2_control_joints>
+                <xacro:insert_block name="ext_axes_ros2_control_joints"/>
+            </ext_axes_ros2_control_joints>
+        </xacro:kuka_ros2_control>
     </xacro:macro>
 </robot>

File: kuka_kr10_description/urdf/kuka.ros2_control.xacro (robot description, xacro)
@@ -2,5 +2,5 @@
 <robot xmlns:xacro="http://www.ros.org/wiki/xacro">
     <xacro:macro name="kuka_ros2_control"
-                 params="name robot_prefix initial_positions_file robot_ip eki_robot_port use_fake_hardware">
+                 params="name robot_prefix initial_positions_file driver_version client_ip client_port mxa_client_port controller_ip mode use_gpio roundtrip_time verify_robot_model **ext_axes_ros2_control_joints">
         <xacro:property name="initial_positions"
                         value="${xacro.load_yaml(initial_positions_file)['initial_positions']}"/>
@@ -10,13 +10,36 @@
             </properties>
             <hardware>
-                <xacro:if value="${use_fake_hardware}">
-                    <plugin>mock_components/GenericSystem</plugin>
+                <xacro:if value="${mode == 'mock'}">
+                    <plugin>kuka_mock_hardware_interface::KukaMockHardwareInterface</plugin>
+                    <param name="cycle_time_ms">4</param>
+                    <param name="roundtrip_time_micro">${roundtrip_time}</param>
+                    <param name="mock_sensor_commands">false</param>
+                    <param name="state_following_offset">0.0</param>
                 </xacro:if>
-                <xacro:unless value="${use_fake_hardware}">
-                    <plugin>kuka_eki_hw_interface/KukaEkiHardwareInterface</plugin>
-                    <param name="robot_ip">${robot_ip}</param>
-                    <param name="eki_robot_port">${eki_robot_port}</param>
-                </xacro:unless>
+                <xacro:if value="${mode == 'hardware'}">
+                    <xacro:if value="${driver_version == 'eki_rsi'}">
+                        <plugin>kuka_rsi_driver::KukaEkiRsiHardwareInterface</plugin>
+                        <param name="controller_ip">${controller_ip}</param>
+                        <param name="client_ip">${client_ip}</param>
+                        <param name="client_port">${client_port}</param>
+                        <param name="name">${name}</param>
+                        <param name="verify_robot_model">${verify_robot_model}</param>
+                    </xacro:if>
+                    <xacro:if value="${driver_version == 'mxa_rsi'}">
+                        <plugin>kuka_rsi_driver::KukaMxaRsiHardwareInterface</plugin>
+                        <param name="controller_ip">${controller_ip}</param>
+                        <param name="client_ip">${client_ip}</param>
+                        <param name="client_port">${client_port}</param>
+                        <param name="mxa_client_port">${mxa_client_port}</param>
+                        <param name="verify_robot_model">${verify_robot_model}</param>
+                    </xacro:if>
+                    <xacro:if value="${driver_version == 'rsi_only'}">
+                        <plugin>kuka_rsi_driver::KukaRSIHardwareInterface</plugin>
+                        <param name="client_ip">${client_ip}</param>
+                        <param name="client_port">${client_port}</param>
+                    </xacro:if>
+                </xacro:if>
             </hardware>
+            <xacro:insert_block name="ext_axes_ros2_control_joints"/>
             <joint name="${robot_prefix}joint_a1">
                 <command_interface name="position"/>
@@ -55,4 +78,11 @@
                 </state_interface>
             </joint>
+            <xacro:if value="${use_gpio}">
+                <xacro:include filename="$(find kuka_rsi_driver)/config/gpio_config.xacro"/>
+                <xacro:gpio_config/>
+            </xacro:if>
+            <xacro:unless value="${use_gpio}">
+                <gpio name="gpio"/>
+            </xacro:unless>
         </ros2_control>
     </xacro:macro>
