Commit message: Changes in the parameters

File: kuka_kr10_description/urdf/kr10r1100sixx.xacro (robot description, xacro)
@@ -4,4 +4,5 @@
     <xacro:arg name="initial_positions_file" default="$(find kuka_kr10_description)/config/initial_positions.yaml"/>
     <xacro:arg name="prefix" default=""/>
+    <xacro:arg name="name" default="kuka_control"/>
     <xacro:arg name="driver_version" default="eki_rsi"/>
     <xacro:arg name="controller_ip" default="10.181.116.41"/>
@@ -14,4 +15,5 @@
     <xacro:arg name="verify_robot_model" default="False"/>
     <xacro:kuka_kr10r1100sixx prefix="$(arg prefix)"
+                              name="$(arg name)"
                               initial_positions_file="$(arg initial_positions_file)"
                               driver_version="$(arg driver_version)"

File: kuka_kr10_description/urdf/kr10r1100sixx_macro.xacro (robot description, xacro)
@@ -4,5 +4,5 @@
     <xacro:include filename="$(find kuka_resources)/urdf/common_materials.xacro"/>
     <xacro:include filename="$(find kuka_kr10_description)/urdf/kuka.ros2_control.xacro"/>
-    <xacro:macro name="kuka_kr10r1100sixx" params="prefix initial_positions_file driver_version client_ip client_port mxa_client_port controller_ip mode use_gpio roundtrip_time verify_robot_model **ext_axes_ros2_control_joints">
+    <xacro:macro name="kuka_kr10r1100sixx" params="prefix name initial_positions_file driver_version client_ip client_port mxa_client_port controller_ip mode use_gpio roundtrip_time verify_robot_model **ext_axes_ros2_control_joints">
         <link name="${prefix}base_link">
             <visual>
@@ -173,5 +173,5 @@
             <origin xyz="0 0 0" rpy="0 ${radians(90)} 0"/>
         </joint>
-        <xacro:kuka_ros2_control name="kuka_control" robot_prefix="${prefix}"
+        <xacro:kuka_ros2_control name="${name}" robot_prefix="${prefix}"
                                  initial_positions_file="${initial_positions_file}"
                                  driver_version="${driver_version}"
@@ -184,5 +184,8 @@
                                  gpio_config="$(find kuka_rsi_driver)/config/gpio_config.xacro"
                                  roundtrip_time="${roundtrip_time}"
-                                 verify_robot_model="${verify_robot_model}">
+                                 verify_robot_model="${verify_robot_model}"
+                                 scheduling_policy="${scheduling_policy}"
+                                 thread_priority="${thread_priority}"
+                                 cpu_affinity="${cpu_affinity}">
             <ext_axes_ros2_control_joints>
                 <xacro:insert_block name="ext_axes_ros2_control_joints"/>

File: kuka_kr10_description/urdf/kuka.ros2_control.xacro (robot description, xacro)
@@ -2,5 +2,5 @@
 <robot xmlns:xacro="http://www.ros.org/wiki/xacro">
     <xacro:macro name="kuka_ros2_control"
-                 params="name robot_prefix initial_positions_file driver_version client_ip client_port mxa_client_port controller_ip mode use_gpio roundtrip_time verify_robot_model
+                 params="name robot_prefix initial_positions_file driver_version client_ip client_port mxa_client_port controller_ip mode use_gpio roundtrip_time verify_robot_model thread_priority:=30 scheduling_policy:='' cpu_affinity:=''
                  gpio_config:='' **ext_axes_ros2_control_joints">
         <xacro:property name="initial_positions"
@@ -9,11 +9,13 @@
             <xacro:property name="gpio_config" value="$(find kuka_rsi_driver)/config/gpio_config.xacro"/>
         </xacro:if>
-        <xacro:property name="scheduling_policy" value="synchronized"/>
-        <xacro:if value="${mode == 'hardware'}">
-            <xacro:property name="scheduling_policy" value="slave"/>
+        <xacro:if value="${scheduling_policy == ''}">
+            <xacro:property name="scheduling_policy" value="synchronized"/>
+            <xacro:if value="${mode == 'hardware'}">
+                <xacro:property name="scheduling_policy" value="slave"/>
+            </xacro:if>
         </xacro:if>
         <ros2_control name="${name}" type="system" is_async="true" rw_rate="250">
             <properties>
-                <async scheduling_policy="${scheduling_policy}" print_warnings="true" thread_priority="30" affinity="[2,3]"/>
+                <async scheduling_policy="${scheduling_policy}" print_warnings="true" thread_priority="${thread_priority}" cpu_affinity="${cpu_affinity}"/>
             </properties>
             <hardware>

Commit message: adjustments in the parameters

File: kuka_kr10_description/urdf/kr10r1100sixx.xacro (robot description, xacro)
@@ -1,4 +1,5 @@
 <?xml version="1.0"?>
 <robot name="kuka_kr10" xmlns:xacro="http://wiki.ros.org/xacro">
+    <!-- TODO: OZ edited -->
     <xacro:include filename="$(find kuka_kr10_description)/urdf/kr10r1100sixx_macro.xacro"/>
     <xacro:arg name="initial_positions_file" default="$(find kuka_kr10_description)/config/initial_positions.yaml"/>
@@ -14,4 +15,7 @@
     <xacro:arg name="roundtrip_time" default="0"/>
     <xacro:arg name="verify_robot_model" default="False"/>
+    <xacro:arg name="scheduling_policy" default=""/>
+    <xacro:arg name="thread_priority" default="30"/>
+    <xacro:arg name="cpu_affinity" default="[2,3]"/>
     <xacro:kuka_kr10r1100sixx prefix="$(arg prefix)"
                               name="$(arg name)"
@@ -25,5 +29,8 @@
                               use_gpio="$(arg use_gpio)"
                               roundtrip_time="$(arg roundtrip_time)"
-                              verify_robot_model="$(arg verify_robot_model)">
+                              verify_robot_model="$(arg verify_robot_model)"
+                              scheduling_policy="$(arg scheduling_policy)"
+                              thread_priority="$(arg thread_priority)"
+                              cpu_affinity="$(arg cpu_affinity)">
         <ext_axes_ros2_control_joints/>
     </xacro:kuka_kr10r1100sixx>

File: kuka_kr10_description/urdf/kr10r1100sixx_macro.xacro (robot description, xacro)
@@ -4,5 +4,6 @@
     <xacro:include filename="$(find kuka_resources)/urdf/common_materials.xacro"/>
     <xacro:include filename="$(find kuka_kr10_description)/urdf/kuka.ros2_control.xacro"/>
-    <xacro:macro name="kuka_kr10r1100sixx" params="prefix name initial_positions_file driver_version client_ip client_port mxa_client_port controller_ip mode use_gpio roundtrip_time verify_robot_model **ext_axes_ros2_control_joints">
+    <!-- TODO: OZ edited -->
+    <xacro:macro name="kuka_kr10r1100sixx" params="prefix name initial_positions_file driver_version client_ip client_port mxa_client_port controller_ip mode use_gpio roundtrip_time verify_robot_model scheduling_policy:='' thread_priority:=30 cpu_affinity:='[2,3]' **ext_axes_ros2_control_joints">
         <link name="${prefix}base_link">
             <visual>

File: kuka_kr10_description/urdf/kuka.ros2_control.xacro (robot description, xacro)
@@ -1,6 +1,7 @@
 <?xml version="1.0"?>
 <robot xmlns:xacro="http://www.ros.org/wiki/xacro">
+    <!-- TODO: OZ edited -->
     <xacro:macro name="kuka_ros2_control"
-                 params="name robot_prefix initial_positions_file driver_version client_ip client_port mxa_client_port controller_ip mode use_gpio roundtrip_time verify_robot_model thread_priority:=30 scheduling_policy:='' cpu_affinity:=''
+                 params="name robot_prefix initial_positions_file driver_version client_ip client_port mxa_client_port controller_ip mode use_gpio roundtrip_time verify_robot_model thread_priority:=30 scheduling_policy:='' cpu_affinity:='[2,3]'
                  gpio_config:='' **ext_axes_ros2_control_joints">
         <xacro:property name="initial_positions"
@@ -17,5 +18,10 @@
         <ros2_control name="${name}" type="system" is_async="true" rw_rate="250">
             <properties>
-                <async scheduling_policy="${scheduling_policy}" print_warnings="true" thread_priority="${thread_priority}" cpu_affinity="${cpu_affinity}"/>
+                <xacro:if value="${cpu_affinity == ''}">
+                    <async scheduling_policy="${scheduling_policy}" print_warnings="true" thread_priority="${thread_priority}"/>
+                </xacro:if>
+                <xacro:unless value="${cpu_affinity == ''}">
+                    <async scheduling_policy="${scheduling_policy}" print_warnings="true" thread_priority="${thread_priority}" affinity="${cpu_affinity}"/>
+                </xacro:unless>
             </properties>
             <hardware>
