Commit message: Explicitly set the scheduling_policy to slave when using real hardware

File: kuka_kr10_description/urdf/kuka.ros2_control.xacro (robot description, xacro)
@@ -5,7 +5,11 @@
         <xacro:property name="initial_positions"
                         value="${xacro.load_yaml(initial_positions_file)['initial_positions']}"/>
+        <xacro:property name="scheduling_policy" value="synchronized"/>
+        <xacro:if value="${mode == 'hardware'}">
+            <xacro:property name="scheduling_policy" value="slave"/>
+        </xacro:if>
         <ros2_control name="${name}" type="system" is_async="true" rw_rate="250">
             <properties>
-                <async scheduling_policy="slave" print_warnings="true" thread_priority="30"/>
+                <async scheduling_policy="${scheduling_policy}" print_warnings="true" thread_priority="30"/>
             </properties>
             <hardware>
