Commit message: Add gpio property

File: kuka_kr10_description/urdf/kr10r1100sixx_macro.xacro (robot description, xacro)
@@ -182,4 +182,5 @@
                                  mode="${mode}"
                                  use_gpio="${use_gpio}"
+                                 gpio_config="$(find kuka_rsi_driver)/config/gpio_config.xacro"
                                  roundtrip_time="${roundtrip_time}"
                                  verify_robot_model="${verify_robot_model}">

File: kuka_kr10_description/urdf/kuka.ros2_control.xacro (robot description, xacro)
@@ -2,7 +2,11 @@
 <robot xmlns:xacro="http://www.ros.org/wiki/xacro">
     <xacro:macro name="kuka_ros2_control"
-                 params="name robot_prefix initial_positions_file driver_version client_ip client_port mxa_client_port controller_ip mode use_gpio roundtrip_time verify_robot_model **ext_axes_ros2_control_joints">
+                 params="name robot_prefix initial_positions_file driver_version client_ip client_port mxa_client_port controller_ip mode use_gpio roundtrip_time verify_robot_model
+                 gpio_config:='' **ext_axes_ros2_control_joints">
         <xacro:property name="initial_positions"
                         value="${xacro.load_yaml(initial_positions_file)['initial_positions']}"/>
+        <xacro:if value="${gpio_config == ''}">
+            <xacro:property name="gpio_config" value="$(find kuka_rsi_driver)/config/gpio_config.xacro"/>
+        </xacro:if>
         <xacro:property name="scheduling_policy" value="synchronized"/>
         <xacro:if value="${mode == 'hardware'}">
@@ -83,5 +87,5 @@
             </joint>
             <xacro:if value="${use_gpio}">
-                <xacro:include filename="$(find kuka_rsi_driver)/config/gpio_config.xacro"/>
+                <xacro:include filename="${gpio_config}"/>
                 <xacro:gpio_config/>
             </xacro:if>

Commit message: add gpio_config arg

File: kuka_kr10_description/urdf/kr10r1100sixx_macro.xacro (robot description, xacro)
@@ -5,5 +5,5 @@
     <xacro:include filename="$(find kuka_kr10_description)/urdf/kuka.ros2_control.xacro"/>
     <!-- TODO: OZ edited -->
-    <xacro:macro name="kuka_kr10r1100sixx" params="prefix name initial_positions_file driver_version client_ip client_port mxa_client_port controller_ip mode use_gpio roundtrip_time verify_robot_model scheduling_policy:='' thread_priority:=30 cpu_affinity:='[2,3]' **ext_axes_ros2_control_joints">
+    <xacro:macro name="kuka_kr10r1100sixx" params="prefix name initial_positions_file driver_version client_ip client_port mxa_client_port controller_ip mode use_gpio roundtrip_time verify_robot_model scheduling_policy:='' thread_priority:=30 cpu_affinity:='[2,3]' gpio_config:='' **ext_axes_ros2_control_joints">
         <link name="${prefix}base_link">
             <visual>
@@ -183,5 +183,5 @@
                                  mode="${mode}"
                                  use_gpio="${use_gpio}"
-                                 gpio_config="$(find kuka_rsi_driver)/config/gpio_config.xacro"
+                                 gpio_config="${gpio_config}"
                                  roundtrip_time="${roundtrip_time}"
                                  verify_robot_model="${verify_robot_model}"

Commit message: add support for motor current

File: kuka_kr10_description/urdf/kr10r1100sixx_macro.xacro (robot description, xacro)
@@ -5,5 +5,5 @@
     <xacro:include filename="$(find kuka_kr10_description)/urdf/kuka.ros2_control.xacro"/>
     <!-- TODO: OZ edited -->
-    <xacro:macro name="kuka_kr10r1100sixx" params="prefix name initial_positions_file driver_version client_ip client_port mxa_client_port controller_ip mode use_gpio roundtrip_time verify_robot_model scheduling_policy:='' thread_priority:=30 cpu_affinity:='[2,3]' gpio_config:='' **ext_axes_ros2_control_joints">
+    <xacro:macro name="kuka_kr10r1100sixx" params="prefix name initial_positions_file driver_version client_ip client_port mxa_client_port controller_ip mode use_gpio roundtrip_time verify_robot_model scheduling_policy:='' thread_priority:=30 cpu_affinity:='[2,3]' gpio_config:='' read_motor_current:=false **ext_axes_ros2_control_joints">
         <link name="${prefix}base_link">
             <visual>
@@ -188,5 +188,6 @@
                                  scheduling_policy="${scheduling_policy}"
                                  thread_priority="${thread_priority}"
-                                 cpu_affinity="${cpu_affinity}">
+                                 cpu_affinity="${cpu_affinity}"
+                                 read_motor_current="${read_motor_current}">
             <ext_axes_ros2_control_joints>
                 <xacro:insert_block name="ext_axes_ros2_control_joints"/>

File: kuka_kr10_description/urdf/kuka.ros2_control.xacro (robot description, xacro)
@@ -4,5 +4,5 @@
     <xacro:macro name="kuka_ros2_control"
                  params="name robot_prefix initial_positions_file driver_version client_ip client_port mxa_client_port controller_ip mode use_gpio roundtrip_time verify_robot_model thread_priority:=30 scheduling_policy:='' cpu_affinity:='[2,3]'
-                 gpio_config:='' **ext_axes_ros2_control_joints">
+                 gpio_config:='' read_motor_current:=false **ext_axes_ros2_control_joints">
         <xacro:property name="initial_positions"
                         value="${xacro.load_yaml(initial_positions_file)['initial_positions']}"/>
@@ -60,4 +60,7 @@
                     <param name="initial_value">${initial_positions['joint_a1']}</param>
                 </state_interface>
+                <xacro:if value="${read_motor_current}">
+                    <state_interface name="current"/>
+                </xacro:if>
             </joint>
             <joint name="${robot_prefix}joint_a2">
@@ -66,4 +69,7 @@
                     <param name="initial_value">${initial_positions['joint_a2']}</param>
                 </state_interface>
+                <xacro:if value="${read_motor_current}">
+                    <state_interface name="current"/>
+                </xacro:if>
             </joint>
             <joint name="${robot_prefix}joint_a3">
@@ -72,4 +78,7 @@
                     <param name="initial_value">${initial_positions['joint_a3']}</param>
                 </state_interface>
+                <xacro:if value="${read_motor_current}">
+                    <state_interface name="current"/>
+                </xacro:if>
             </joint>
             <joint name="${robot_prefix}joint_a4">
@@ -78,4 +87,7 @@
                     <param name="initial_value">${initial_positions['joint_a4']}</param>
                 </state_interface>
+                <xacro:if value="${read_motor_current}">
+                    <state_interface name="current"/>
+                </xacro:if>
             </joint>
             <joint name="${robot_prefix}joint_a5">
@@ -84,4 +96,7 @@
                     <param name="initial_value">${initial_positions['joint_a5']}</param>
                 </state_interface>
+                <xacro:if value="${read_motor_current}">
+                    <state_interface name="current"/>
+                </xacro:if>
             </joint>
             <joint name="${robot_prefix}joint_a6">
@@ -90,4 +105,7 @@
                     <param name="initial_value">${initial_positions['joint_a6']}</param>
                 </state_interface>
+                <xacro:if value="${read_motor_current}">
+                    <state_interface name="current"/>
+                </xacro:if>
             </joint>
             <xacro:if value="${use_gpio}">

Commit message: RSol RIst read cartesian pose

File: kuka_kr10_description/urdf/kr10r1100sixx_macro.xacro (robot description, xacro)
@@ -5,5 +5,5 @@
     <xacro:include filename="$(find kuka_kr10_description)/urdf/kuka.ros2_control.xacro"/>
     <!-- TODO: OZ edited -->
-    <xacro:macro name="kuka_kr10r1100sixx" params="prefix name initial_positions_file driver_version client_ip client_port mxa_client_port controller_ip mode use_gpio roundtrip_time verify_robot_model scheduling_policy:='' thread_priority:=30 cpu_affinity:='[2,3]' gpio_config:='' read_motor_current:=false **ext_axes_ros2_control_joints">
+    <xacro:macro name="kuka_kr10r1100sixx" params="prefix name initial_positions_file driver_version client_ip client_port mxa_client_port controller_ip mode use_gpio roundtrip_time verify_robot_model scheduling_policy:='' thread_priority:=30 cpu_affinity:='[2,3]' gpio_config:='' read_motor_current:=false read_cartesian_setpoint:=false read_cartesian_pose:=false **ext_axes_ros2_control_joints">
         <link name="${prefix}base_link">
             <visual>
@@ -189,5 +189,7 @@
                                  thread_priority="${thread_priority}"
                                  cpu_affinity="${cpu_affinity}"
-                                 read_motor_current="${read_motor_current}">
+                                 read_motor_current="${read_motor_current}"
+                                 read_cartesian_setpoint="${read_cartesian_setpoint}"
+                                 read_cartesian_pose="${read_cartesian_pose}">
             <ext_axes_ros2_control_joints>
                 <xacro:insert_block name="ext_axes_ros2_control_joints"/>

File: kuka_kr10_description/urdf/kuka.ros2_control.xacro (robot description, xacro)
@@ -4,5 +4,5 @@
     <xacro:macro name="kuka_ros2_control"
                  params="name robot_prefix initial_positions_file driver_version client_ip client_port mxa_client_port controller_ip mode use_gpio roundtrip_time verify_robot_model thread_priority:=30 scheduling_policy:='' cpu_affinity:='[2,3]'
-                 gpio_config:='' read_motor_current:=false **ext_axes_ros2_control_joints">
+                 gpio_config:='' read_motor_current:=false read_cartesian_setpoint:=false read_cartesian_pose:=false **ext_axes_ros2_control_joints">
         <xacro:property name="initial_positions"
                         value="${xacro.load_yaml(initial_positions_file)['initial_positions']}"/>
@@ -116,4 +116,24 @@
                 <gpio name="gpio"/>
             </xacro:unless>
+            <xacro:if value="${read_cartesian_setpoint}">
+                <sensor name="cartesian_setpoint">
+                    <state_interface name="x"/>
+                    <state_interface name="y"/>
+                    <state_interface name="z"/>
+                    <state_interface name="a"/>
+                    <state_interface name="b"/>
+                    <state_interface name="c"/>
+                </sensor>
+            </xacro:if>
+            <xacro:if value="${read_cartesian_pose}">
+                <sensor name="cartesian_pose">
+                    <state_interface name="x"/>
+                    <state_interface name="y"/>
+                    <state_interface name="z"/>
+                    <state_interface name="a"/>
+                    <state_interface name="b"/>
+                    <state_interface name="c"/>
+                </sensor>
+            </xacro:if>
         </ros2_control>
     </xacro:macro>

Commit message: progress status and speed scaling added

File: kuka_kr10_description/urdf/kr10r1100sixx_macro.xacro (robot description, xacro)
@@ -5,5 +5,5 @@
     <xacro:include filename="$(find kuka_kr10_description)/urdf/kuka.ros2_control.xacro"/>
     <!-- TODO: OZ edited -->
-    <xacro:macro name="kuka_kr10r1100sixx" params="prefix name initial_positions_file driver_version client_ip client_port mxa_client_port controller_ip mode use_gpio roundtrip_time verify_robot_model scheduling_policy:='' thread_priority:=30 cpu_affinity:='[2,3]' gpio_config:='' read_motor_current:=false read_cartesian_setpoint:=false read_cartesian_pose:=false **ext_axes_ros2_control_joints">
+    <xacro:macro name="kuka_kr10r1100sixx" params="prefix name initial_positions_file driver_version client_ip client_port mxa_client_port controller_ip mode use_gpio roundtrip_time verify_robot_model scheduling_policy:='' thread_priority:=30 cpu_affinity:='[2,3]' gpio_config:='' read_motor_current:=false read_gear_torque:=false read_cartesian_setpoint:=false read_cartesian_pose:=false read_robot_status:=false **ext_axes_ros2_control_joints">
         <link name="${prefix}base_link">
             <visual>
@@ -190,6 +190,8 @@
                                  cpu_affinity="${cpu_affinity}"
                                  read_motor_current="${read_motor_current}"
+                                 read_gear_torque="${read_gear_torque}"
                                  read_cartesian_setpoint="${read_cartesian_setpoint}"
-                                 read_cartesian_pose="${read_cartesian_pose}">
+                                 read_cartesian_pose="${read_cartesian_pose}"
+                                 read_robot_status="${read_robot_status}">
             <ext_axes_ros2_control_joints>
                 <xacro:insert_block name="ext_axes_ros2_control_joints"/>

File: kuka_kr10_description/urdf/kuka.ros2_control.xacro (robot description, xacro)
@@ -4,5 +4,5 @@
     <xacro:macro name="kuka_ros2_control"
                  params="name robot_prefix initial_positions_file driver_version client_ip client_port mxa_client_port controller_ip mode use_gpio roundtrip_time verify_robot_model thread_priority:=30 scheduling_policy:='' cpu_affinity:='[2,3]'
-                 gpio_config:='' read_motor_current:=false read_cartesian_setpoint:=false read_cartesian_pose:=false **ext_axes_ros2_control_joints">
+                 gpio_config:='' read_motor_current:=false read_gear_torque:=false read_cartesian_setpoint:=false read_cartesian_pose:=false read_robot_status:=false **ext_axes_ros2_control_joints">
         <xacro:property name="initial_positions"
                         value="${xacro.load_yaml(initial_positions_file)['initial_positions']}"/>
@@ -63,4 +63,7 @@
                     <state_interface name="current"/>
                 </xacro:if>
+                <xacro:if value="${read_gear_torque}">
+                    <state_interface name="torque"/>
+                </xacro:if>
             </joint>
             <joint name="${robot_prefix}joint_a2">
@@ -71,4 +74,7 @@
                 <xacro:if value="${read_motor_current}">
                     <state_interface name="current"/>
+                </xacro:if>
+                <xacro:if value="${read_gear_torque}">
+                    <state_interface name="torque"/>
                 </xacro:if>
             </joint>
@@ -81,4 +87,7 @@
                     <state_interface name="current"/>
                 </xacro:if>
+                <xacro:if value="${read_gear_torque}">
+                    <state_interface name="torque"/>
+                </xacro:if>
             </joint>
             <joint name="${robot_prefix}joint_a4">
@@ -89,4 +98,7 @@
                 <xacro:if value="${read_motor_current}">
                     <state_interface name="current"/>
+                </xacro:if>
+                <xacro:if value="${read_gear_torque}">
+                    <state_interface name="torque"/>
                 </xacro:if>
             </joint>
@@ -99,4 +111,7 @@
                     <state_interface name="current"/>
                 </xacro:if>
+                <xacro:if value="${read_gear_torque}">
+                    <state_interface name="torque"/>
+                </xacro:if>
             </joint>
             <joint name="${robot_prefix}joint_a6">
@@ -107,4 +122,7 @@
                 <xacro:if value="${read_motor_current}">
                     <state_interface name="current"/>
+                </xacro:if>
+                <xacro:if value="${read_gear_torque}">
+                    <state_interface name="torque"/>
                 </xacro:if>
             </joint>
@@ -136,4 +154,10 @@
                 </sensor>
             </xacro:if>
+            <xacro:if value="${read_robot_status}">
+                <sensor name="robot_status">
+                    <state_interface name="program_state"/>
+                    <state_interface name="speed_scaling_factor"/>
+                </sensor>
+            </xacro:if>
         </ros2_control>
     </xacro:macro>
