Commit message: Expose the cpu_affinity and gpio_config in ros2_control XACROs

File: kuka_agilus_support/urdf/kr_agilus_ros2_control_macro.xacro (robot description, xacro)
@@ -1,5 +1,8 @@
 <?xml version="1.0" encoding="UTF-8"?>
 <robot xmlns:xacro="http://www.ros.org/wiki/xacro">
-  <xacro:macro name="kuka_agilus_ros2_control" params="name driver_version client_ip client_port mxa_client_port controller_ip prefix mode use_gpio roundtrip_time verify_robot_model **ext_axes_ros2_control_joints">
+  <xacro:macro name="kuka_agilus_ros2_control" params="name driver_version client_ip client_port mxa_client_port controller_ip prefix mode use_gpio roundtrip_time verify_robot_model gpio_config:='' **ext_axes_ros2_control_joints">
+    <xacro:if value="${gpio_config == ''}">
+      <xacro:property name="gpio_config" value="$(find kuka_rsi_driver)/config/gpio_config.xacro"/>
+    </xacro:if>
     <!-- gazebo -->
     <xacro:if value="${mode == 'gazebo'}">
@@ -10,5 +13,5 @@
     <ros2_control name="${name}" type="system" is_async="true" rw_rate="250">
       <properties>
-        <async scheduling_policy="slave" print_warnings="true" thread_priority="30"/>
+        <async scheduling_policy="slave" print_warnings="true" thread_priority="30" affinity="[2,3]"/>
       </properties>
       <hardware>
@@ -85,5 +88,5 @@
       </joint>
       <xacro:if value="${use_gpio}">
-        <xacro:include filename="$(find kuka_rsi_driver)/config/gpio_config.xacro"/>
+        <xacro:include filename="${gpio_config}"/>
         <xacro:gpio_config/>
       </xacro:if>

File: kuka_fortec_support/urdf/kr_fortec_ros2_control_macro.xacro (robot description, xacro)
@@ -1,5 +1,8 @@
 <?xml version="1.0" encoding="UTF-8"?>
 <robot xmlns:xacro="http://www.ros.org/wiki/xacro">
-  <xacro:macro name="kuka_fortec_ros2_control" params="name driver_version client_ip client_port mxa_client_port controller_ip prefix mode use_gpio roundtrip_time verify_robot_model **ext_axes_ros2_control_joints">
+  <xacro:macro name="kuka_fortec_ros2_control" params="name driver_version client_ip client_port mxa_client_port controller_ip prefix mode use_gpio roundtrip_time verify_robot_model gpio_config:='' **ext_axes_ros2_control_joints">
+    <xacro:if value="${gpio_config == ''}">
+      <xacro:property name="gpio_config" value="$(find kuka_rsi_driver)/config/gpio_config.xacro"/>
+    </xacro:if>
     <!-- gazebo -->
     <xacro:if value="${mode == 'gazebo'}">
@@ -14,5 +17,5 @@
     <ros2_control name="${name}" type="system" is_async="true" rw_rate="250">
       <properties>
-        <async scheduling_policy="${scheduling_policy}" print_warnings="true" thread_priority="30"/>
+        <async scheduling_policy="${scheduling_policy}" print_warnings="true" thread_priority="30" affinity="[2,3]"/>
       </properties>
       <hardware>
@@ -89,5 +92,5 @@
       </joint>
       <xacro:if value="${use_gpio}">
-        <xacro:include filename="$(find kuka_rsi_driver)/config/gpio_config.xacro"/>
+        <xacro:include filename="${gpio_config}"/>
         <xacro:gpio_config/>
       </xacro:if>
