Commit message: Only set the affinity value for the concerned models kr10_r1100_sixx and kr340_r3400_2

File: kuka_agilus_support/urdf/kr10_r1100_sixx.xacro (robot description, xacro)
@@ -7,4 +7,6 @@
     <xacro:arg name="mode" default="hardware"/>
     <xacro:arg name="use_gpio" default="false"/>
+    <xacro:arg name="gpio_config" default=""/>
+    <xacro:arg name="affinity" default="[2,3]"/>
     <xacro:arg name="roundtrip_time" default="0"/>
     <xacro:arg name="client_ip" default="0.0.0.0"/>
@@ -20,5 +22,5 @@
     <xacro:arg name="pitch" default="0"/>
     <xacro:arg name="yaw" default="0"/>
-    <xacro:kuka_agilus_ros2_control name="$(arg prefix)kr10_r1100_sixx" driver_version="$(arg driver_version)" client_ip="$(arg client_ip)" client_port="$(arg client_port)" mxa_client_port="$(arg mxa_client_port)" controller_ip="$(arg controller_ip)" prefix="$(arg prefix)" mode="$(arg mode)" use_gpio="$(arg use_gpio)" roundtrip_time="$(arg roundtrip_time)" verify_robot_model="$(arg verify_robot_model)">
+    <xacro:kuka_agilus_ros2_control name="$(arg prefix)kr10_r1100_sixx" driver_version="$(arg driver_version)" client_ip="$(arg client_ip)" client_port="$(arg client_port)" mxa_client_port="$(arg mxa_client_port)" controller_ip="$(arg controller_ip)" prefix="$(arg prefix)" mode="$(arg mode)" use_gpio="$(arg use_gpio)" gpio_config="$(arg gpio_config)" affinity="$(arg affinity)" roundtrip_time="$(arg roundtrip_time)" verify_robot_model="$(arg verify_robot_model)">
         <ext_axes_ros2_control_joints/>
     </xacro:kuka_agilus_ros2_control>

File: kuka_agilus_support/urdf/kr_agilus_ros2_control_macro.xacro (robot description, xacro)
@@ -1,5 +1,5 @@
 <?xml version="1.0" encoding="UTF-8"?>
 <robot xmlns:xacro="http://www.ros.org/wiki/xacro">
-  <xacro:macro name="kuka_agilus_ros2_control" params="name driver_version client_ip client_port mxa_client_port controller_ip prefix mode use_gpio roundtrip_time verify_robot_model gpio_config:='' **ext_axes_ros2_control_joints">
+  <xacro:macro name="kuka_agilus_ros2_control" params="name driver_version client_ip client_port mxa_client_port controller_ip prefix mode use_gpio roundtrip_time verify_robot_model gpio_config:='' affinity:='' **ext_axes_ros2_control_joints">
     <xacro:if value="${gpio_config == ''}">
       <xacro:property name="gpio_config" value="$(find kuka_rsi_driver)/config/gpio_config.xacro"/>
@@ -13,5 +13,10 @@
     <ros2_control name="${name}" type="system" is_async="true" rw_rate="250">
       <properties>
-        <async scheduling_policy="slave" print_warnings="true" thread_priority="30" affinity="[2,3]"/>
+        <xacro:if value="${affinity == ''}">
+          <async scheduling_policy="slave" print_warnings="true" thread_priority="30"/>
+        </xacro:if>
+        <xacro:unless value="${affinity == ''}">
+          <async scheduling_policy="slave" print_warnings="true" thread_priority="30" affinity="${affinity}"/>
+        </xacro:unless>
       </properties>
       <hardware>

File: kuka_fortec_support/urdf/kr340_r3400_2.urdf.xacro (robot description, xacro)
@@ -8,4 +8,6 @@
   <xacro:arg name="mode" default="hardware"/>
   <xacro:arg name="use_gpio" default="false"/>
+  <xacro:arg name="gpio_config" default=""/>
+  <xacro:arg name="affinity" default="[2,3]"/>
   <xacro:arg name="roundtrip_time" default="0"/>
   <xacro:arg name="client_ip" default="0.0.0.0"/>
@@ -21,5 +23,5 @@
   <xacro:arg name="pitch" default="0"/>
   <xacro:arg name="yaw" default="0"/>
-  <xacro:kuka_fortec_ros2_control name="$(arg prefix)kr340_r3400_2" driver_version="$(arg driver_version)" client_ip="$(arg client_ip)" client_port="$(arg client_port)" mxa_client_port="$(arg mxa_client_port)" controller_ip="$(arg controller_ip)" prefix="$(arg prefix)" mode="$(arg mode)" use_gpio="$(arg use_gpio)" roundtrip_time="$(arg roundtrip_time)" verify_robot_model="$(arg verify_robot_model)">
+  <xacro:kuka_fortec_ros2_control name="$(arg prefix)kr340_r3400_2" driver_version="$(arg driver_version)" client_ip="$(arg client_ip)" client_port="$(arg client_port)" mxa_client_port="$(arg mxa_client_port)" controller_ip="$(arg controller_ip)" prefix="$(arg prefix)" mode="$(arg mode)" use_gpio="$(arg use_gpio)" gpio_config="$(arg gpio_config)" affinity="$(arg affinity)" roundtrip_time="$(arg roundtrip_time)" verify_robot_model="$(arg verify_robot_model)">
     <ext_axes_ros2_control_joints/>
   </xacro:kuka_fortec_ros2_control>

File: kuka_fortec_support/urdf/kr_fortec_ros2_control_macro.xacro (robot description, xacro)
@@ -1,5 +1,5 @@
 <?xml version="1.0" encoding="UTF-8"?>
 <robot xmlns:xacro="http://www.ros.org/wiki/xacro">
-  <xacro:macro name="kuka_fortec_ros2_control" params="name driver_version client_ip client_port mxa_client_port controller_ip prefix mode use_gpio roundtrip_time verify_robot_model gpio_config:='' **ext_axes_ros2_control_joints">
+  <xacro:macro name="kuka_fortec_ros2_control" params="name driver_version client_ip client_port mxa_client_port controller_ip prefix mode use_gpio roundtrip_time verify_robot_model gpio_config:='' affinity:='' **ext_axes_ros2_control_joints">
     <xacro:if value="${gpio_config == ''}">
       <xacro:property name="gpio_config" value="$(find kuka_rsi_driver)/config/gpio_config.xacro"/>
@@ -17,5 +17,10 @@
     <ros2_control name="${name}" type="system" is_async="true" rw_rate="250">
       <properties>
-        <async scheduling_policy="${scheduling_policy}" print_warnings="true" thread_priority="30" affinity="[2,3]"/>
+        <xacro:if value="${affinity == ''}">
+          <async scheduling_policy="${scheduling_policy}" print_warnings="true" thread_priority="30"/>
+        </xacro:if>
+        <xacro:unless value="${affinity == ''}">
+          <async scheduling_policy="${scheduling_policy}" print_warnings="true" thread_priority="30" affinity="${affinity}"/>
+        </xacro:unless>
       </properties>
       <hardware>

Commit message: Update the async parameters of the agilus family

File: kuka_agilus_support/urdf/kr10_r1100_sixx.xacro (robot description, xacro)
@@ -7,6 +7,8 @@
     <xacro:arg name="mode" default="hardware"/>
     <xacro:arg name="use_gpio" default="false"/>
-    <xacro:arg name="gpio_config" default=""/>
-    <xacro:arg name="affinity" default="[2,3]"/>
+    <xacro:arg name="is_async" default="true"/>
+    <xacro:arg name="scheduling_policy" default="slave"/>
+    <xacro:arg name="thread_priority" default="30"/>
+    <xacro:arg name="cpu_affinity" default="[2,3]"/>
     <xacro:arg name="roundtrip_time" default="0"/>
     <xacro:arg name="client_ip" default="0.0.0.0"/>
@@ -22,5 +24,5 @@
     <xacro:arg name="pitch" default="0"/>
     <xacro:arg name="yaw" default="0"/>
-    <xacro:kuka_agilus_ros2_control name="$(arg prefix)kr10_r1100_sixx" driver_version="$(arg driver_version)" client_ip="$(arg client_ip)" client_port="$(arg client_port)" mxa_client_port="$(arg mxa_client_port)" controller_ip="$(arg controller_ip)" prefix="$(arg prefix)" mode="$(arg mode)" use_gpio="$(arg use_gpio)" gpio_config="$(arg gpio_config)" affinity="$(arg affinity)" roundtrip_time="$(arg roundtrip_time)" verify_robot_model="$(arg verify_robot_model)">
+    <xacro:kuka_agilus_ros2_control name="$(arg prefix)kr10_r1100_sixx" driver_version="$(arg driver_version)" client_ip="$(arg client_ip)" client_port="$(arg client_port)" mxa_client_port="$(arg mxa_client_port)" controller_ip="$(arg controller_ip)" prefix="$(arg prefix)" mode="$(arg mode)" use_gpio="$(arg use_gpio)" is_async="$(arg is_async)" scheduling_policy="$(arg scheduling_policy)" thread_priority="$(arg thread_priority)" cpu_affinity="$(arg cpu_affinity)" roundtrip_time="$(arg roundtrip_time)" verify_robot_model="$(arg verify_robot_model)">
         <ext_axes_ros2_control_joints/>
     </xacro:kuka_agilus_ros2_control>

File: kuka_agilus_support/urdf/kr_agilus_ros2_control_macro.xacro (robot description, xacro)
@@ -1,8 +1,21 @@
 <?xml version="1.0" encoding="UTF-8"?>
 <robot xmlns:xacro="http://www.ros.org/wiki/xacro">
-  <xacro:macro name="kuka_agilus_ros2_control" params="name driver_version client_ip client_port mxa_client_port controller_ip prefix mode use_gpio roundtrip_time verify_robot_model gpio_config:='' affinity:='' **ext_axes_ros2_control_joints">
-    <xacro:if value="${gpio_config == ''}">
-      <xacro:property name="gpio_config" value="$(find kuka_rsi_driver)/config/gpio_config.xacro"/>
-    </xacro:if>
+  <xacro:macro name="kuka_agilus_ros2_control"
+              params="name
+              driver_version
+              client_ip
+              client_port
+              mxa_client_port
+              controller_ip
+              prefix
+              mode
+              use_gpio
+              roundtrip_time
+              verify_robot_model
+              **ext_axes_ros2_control_joints
+              is_async:=false
+              scheduling_policy:=detached
+              thread_priority:=30
+              cpu_affinity:=''">
     <!-- gazebo -->
     <xacro:if value="${mode == 'gazebo'}">
@@ -11,13 +24,10 @@
     </xacro:if>
     <!-- ros2 control -->
-    <ros2_control name="${name}" type="system" is_async="true" rw_rate="250">
-      <properties>
-        <xacro:if value="${affinity == ''}">
-          <async scheduling_policy="slave" print_warnings="true" thread_priority="30"/>
+    <ros2_control name="${name}" type="system" is_async="${is_async}" rw_rate="250">
+       <xacro:if value="${is_async}">
+            <properties>
+                <async scheduling_policy="${scheduling_policy}" print_warnings="true" thread_priority="${thread_priority}" affinity="${cpu_affinity}"/>
+            </properties>
         </xacro:if>
-        <xacro:unless value="${affinity == ''}">
-          <async scheduling_policy="slave" print_warnings="true" thread_priority="30" affinity="${affinity}"/>
-        </xacro:unless>
-      </properties>
       <hardware>
         <xacro:if value="${mode == 'mock'}">
@@ -93,5 +103,5 @@
       </joint>
       <xacro:if value="${use_gpio}">
-        <xacro:include filename="${gpio_config}"/>
+        <xacro:include filename="$(find kuka_rsi_driver)/config/gpio_config.xacro"/>
         <xacro:gpio_config/>
       </xacro:if>
