Commit message: Apply pre-commit XML formatting
Co-Authored-By: Claude Sonnet 5 <noreply@anthropic.com>

File: kuka_agilus_support/urdf/kr10_r1100_sixx.xacro (robot description, xacro)
@@ -1,41 +1,41 @@
 <?xml version="1.0"?>
-<robot name="kuka_kr10" xmlns:xacro="http://wiki.ros.org/xacro">
-    <xacro:include filename="$(find kuka_agilus_support)/urdf/kr10_r1100_sixx_macro.xacro"/>
-    <xacro:include filename="$(find kuka_agilus_support)/urdf/kr_agilus_ros2_control_macro.xacro"/>
-    <!-- Read additional arguments  -->
-    <xacro:arg name="driver_version" default="rsi_only"/>
-    <xacro:arg name="mode" default="hardware"/>
-    <xacro:arg name="use_gpio" default="false"/>
-    <xacro:arg name="gpio_config" default=""/>
-    <xacro:arg name="scheduling_policy" default="detached"/>
-    <xacro:arg name="roundtrip_time" default="0"/>
-    <xacro:arg name="client_ip" default="0.0.0.0"/>
-    <xacro:arg name="client_port" default="59152"/>
-    <xacro:arg name="mxa_client_port" default="1337"/>
-    <xacro:arg name="controller_ip" default="0.0.0.0"/>
-    <xacro:arg name="verify_robot_model" default="true"/>
-    <xacro:arg name="prefix" default=""/>
-    <xacro:arg name="is_async" default="false"/>
-    <xacro:arg name="async_thread_priority" default="69"/>
-    <xacro:arg name="async_affinity" default="[]"/>
-    <xacro:arg name="x" default="0"/>
-    <xacro:arg name="y" default="0"/>
-    <xacro:arg name="z" default="0"/>
-    <xacro:arg name="roll" default="0"/>
-    <xacro:arg name="pitch" default="0"/>
-    <xacro:arg name="yaw" default="0"/>
-    <xacro:arg name="rsi_xml_config_file" default=""/>
-    <xacro:kuka_agilus_ros2_control name="$(arg prefix)kr10_r1100_sixx" driver_version="$(arg driver_version)" client_ip="$(arg client_ip)" client_port="$(arg client_port)" mxa_client_port="$(arg mxa_client_port)" controller_ip="$(arg controller_ip)" prefix="$(arg prefix)" mode="$(arg mode)" use_gpio="$(arg use_gpio)" gpio_config="$(arg gpio_config)" roundtrip_time="$(arg roundtrip_time)" verify_robot_model="$(arg verify_robot_model)" rsi_xml_config_file="$(arg rsi_xml_config_file)" is_async="$(arg is_async)" scheduling_policy="$(arg scheduling_policy)" async_thread_priority="$(arg async_thread_priority)" async_affinity="$(arg async_affinity)">
-        <ext_axes_ros2_control_joints/>
-    </xacro:kuka_agilus_ros2_control>
-    <!-- world link -->
-    <link name="world"/>
-    <!-- robot links, joints -->
-    <xacro:kuka_kr10_r1100_sixx_robot prefix="$(arg prefix)" package_name="kuka_agilus_support"/>
-    <!-- default world - base_link joint -->
-    <joint name="$(arg prefix)world-base_link" type="fixed">
-        <parent link="world"/>
-        <child link="$(arg prefix)base_link"/>
-        <origin xyz="$(arg x) $(arg y) $(arg z)" rpy="$(arg roll) $(arg pitch) $(arg yaw)"/>
-    </joint>
+<robot xmlns:xacro="http://wiki.ros.org/xacro" name="kuka_kr10">
+  <xacro:include filename="$(find kuka_agilus_support)/urdf/kr10_r1100_sixx_macro.xacro"/>
+  <xacro:include filename="$(find kuka_agilus_support)/urdf/kr_agilus_ros2_control_macro.xacro"/>
+  <!-- Read additional arguments  -->
+  <xacro:arg name="driver_version" default="rsi_only"/>
+  <xacro:arg name="mode" default="hardware"/>
+  <xacro:arg name="use_gpio" default="false"/>
+  <xacro:arg name="gpio_config" default=""/>
+  <xacro:arg name="scheduling_policy" default="detached"/>
+  <xacro:arg name="roundtrip_time" default="0"/>
+  <xacro:arg name="client_ip" default="0.0.0.0"/>
+  <xacro:arg name="client_port" default="59152"/>
+  <xacro:arg name="mxa_client_port" default="1337"/>
+  <xacro:arg name="controller_ip" default="0.0.0.0"/>
+  <xacro:arg name="verify_robot_model" default="true"/>
+  <xacro:arg name="prefix" default=""/>
+  <xacro:arg name="is_async" default="false"/>
+  <xacro:arg name="async_thread_priority" default="69"/>
+  <xacro:arg name="async_affinity" default="[]"/>
+  <xacro:arg name="x" default="0"/>
+  <xacro:arg name="y" default="0"/>
+  <xacro:arg name="z" default="0"/>
+  <xacro:arg name="roll" default="0"/>
+  <xacro:arg name="pitch" default="0"/>
+  <xacro:arg name="yaw" default="0"/>
+  <xacro:arg name="rsi_xml_config_file" default=""/>
+  <xacro:kuka_agilus_ros2_control name="$(arg prefix)kr10_r1100_sixx" driver_version="$(arg driver_version)" client_ip="$(arg client_ip)" client_port="$(arg client_port)" mxa_client_port="$(arg mxa_client_port)" controller_ip="$(arg controller_ip)" prefix="$(arg prefix)" mode="$(arg mode)" use_gpio="$(arg use_gpio)" gpio_config="$(arg gpio_config)" roundtrip_time="$(arg roundtrip_time)" verify_robot_model="$(arg verify_robot_model)" rsi_xml_config_file="$(arg rsi_xml_config_file)" is_async="$(arg is_async)" scheduling_policy="$(arg scheduling_policy)" async_thread_priority="$(arg async_thread_priority)" async_affinity="$(arg async_affinity)">
+    <ext_axes_ros2_control_joints/>
+  </xacro:kuka_agilus_ros2_control>
+  <!-- world link -->
+  <link name="world"/>
+  <!-- robot links, joints -->
+  <xacro:kuka_kr10_r1100_sixx_robot prefix="$(arg prefix)" package_name="kuka_agilus_support"/>
+  <!-- default world - base_link joint -->
+  <joint name="$(arg prefix)world-base_link" type="fixed">
+    <parent link="world"/>
+    <child link="$(arg prefix)base_link"/>
+    <origin xyz="$(arg x) $(arg y) $(arg z)" rpy="$(arg roll) $(arg pitch) $(arg yaw)"/>
+  </joint>
 </robot>

File: kuka_agilus_support/urdf/kr10_r1100_sixx_macro.xacro (robot description, xacro)
@@ -1,171 +1,171 @@
 <?xml version="1.0"?>
 <robot xmlns:xacro="http://wiki.ros.org/xacro">
-    <xacro:include filename="$(find kuka_resources)/urdf/common_constants.xacro"/>
-    <xacro:include filename="$(find kuka_resources)/urdf/common_materials.xacro"/>
-    <xacro:macro name="kuka_kr10_r1100_sixx_robot" params="prefix package_name">
+  <xacro:include filename="$(find kuka_resources)/urdf/common_constants.xacro"/>
+  <xacro:include filename="$(find kuka_resources)/urdf/common_materials.xacro"/>
+  <xacro:macro name="kuka_kr10_r1100_sixx_robot" params="prefix package_name">
     <link name="${prefix}base"/>
     <link name="${prefix}base_link">
-        <visual>
-            <origin xyz="0 0 0" rpy="0 0 0"/>
-            <geometry>
-                <mesh filename="package://${package_name}/meshes/kr10_r1100_sixx/visual/base_link.stl"/>
-            </geometry>
-            <xacro:material_kuka_black/>
-        </visual>
-        <collision>
-            <origin xyz="0 0 0" rpy="0 0 0"/>
-            <geometry>
-                <mesh filename="package://${package_name}/meshes/kr10_r1100_sixx/collision/base_link.stl"/>
-            </geometry>
-        </collision>
+      <visual>
+        <origin xyz="0 0 0" rpy="0 0 0"/>
+        <geometry>
+          <mesh filename="package://${package_name}/meshes/kr10_r1100_sixx/visual/base_link.stl"/>
+        </geometry>
+        <xacro:material_kuka_black/>
+      </visual>
+      <collision>
+        <origin xyz="0 0 0" rpy="0 0 0"/>
+        <geometry>
+          <mesh filename="package://${package_name}/meshes/kr10_r1100_sixx/collision/base_link.stl"/>
+        </geometry>
+      </collision>
     </link>
     <link name="${prefix}flange"/>
     <link name="${prefix}link_1">
-        <visual>
-            <origin xyz="0 0 0" rpy="0 0 0"/>
-            <geometry>
-                <mesh filename="package://${package_name}/meshes/kr10_r1100_sixx/visual/link_1.stl"/>
-            </geometry>
-            <xacro:material_kuka_orange/>
-        </visual>
-        <collision>
-            <origin xyz="0 0 0" rpy="0 0 0"/>
-            <geometry>
-                <mesh filename="package://${package_name}/meshes/kr10_r1100_sixx/collision/link_1.stl"/>
-            </geometry>
-        </collision>
+      <visual>
+        <origin xyz="0 0 0" rpy="0 0 0"/>
+        <geometry>
+          <mesh filename="package://${package_name}/meshes/kr10_r1100_sixx/visual/link_1.stl"/>
+        </geometry>
+        <xacro:material_kuka_orange/>
+      </visual>
+      <collision>
+        <origin xyz="0 0 0" rpy="0 0 0"/>
+        <geometry>
+          <mesh filename="package://${package_name}/meshes/kr10_r1100_sixx/collision/link_1.stl"/>
+        </geometry>
+      </collision>
     </link>
     <link name="${prefix}link_2">
-        <visual>
-            <origin xyz="0 0 0" rpy="0 0 0"/>
-            <geometry>
-                <mesh filename="package://${package_name}/meshes/kr10_r1100_sixx/visual/link_2.stl"/>
-            </geometry>
-            <xacro:material_kuka_orange/>
-        </visual>
-        <collision>
-            <origin xyz="0 0 0" rpy="0 0 0"/>
-            <geometry>
-                <mesh filename="package://${package_name}/meshes/kr10_r1100_sixx/collision/link_2.stl"/>
-            </geometry>
-        </collision>
+      <visual>
+        <origin xyz="0 0 0" rpy="0 0 0"/>
+        <geometry>
+          <mesh filename="package://${package_name}/meshes/kr10_r1100_sixx/visual/link_2.stl"/>
+        </geometry>
+        <xacro:material_kuka_orange/>
+      </visual>
+      <collision>
+        <origin xyz="0 0 0" rpy="0 0 0"/>
+        <geometry>
+          <mesh filename="package://${package_name}/meshes/kr10_r1100_sixx/collision/link_2.stl"/>
+        </geometry>
+      </collision>
     </link>
     <link name="${prefix}link_3">
-        <visual>
-            <origin xyz="0 0 0" rpy="0 0 0"/>
-            <geometry>
-                <mesh filename="package://${package_name}/meshes/kr10_r1100_sixx/visual/link_3.stl"/>
-            </geometry>
-            <xacro:material_kuka_orange/>
-        </visual>
-        <collision>
-            <origin xyz="0 0 0" rpy="0 0 0"/>
-            <geometry>
-                <mesh filename="package://${package_name}/meshes/kr10_r1100_sixx/collision/link_3.stl"/>
-            </geometry>
-        </collision>
+      <visual>
+        <origin xyz="0 0 0" rpy="0 0 0"/>
+        <geometry>
+          <mesh filename="package://${package_name}/meshes/kr10_r1100_sixx/visual/link_3.stl"/>
+        </geometry>
+        <xacro:material_kuka_orange/>
+      </visual>
+      <collision>
+        <origin xyz="0 0 0" rpy="0 0 0"/>
+        <geometry>
+          <mesh filename="package://${package_name}/meshes/kr10_r1100_sixx/collision/link_3.stl"/>
+        </geometry>
+      </collision>
     </link>
     <link name="${prefix}link_4">
-        <visual>
-            <origin xyz="0 0 0" rpy="0 0 0"/>
-            <geometry>
-                <mesh filename="package://${package_name}/meshes/kr10_r1100_sixx/visual/link_4.stl"/>
-            </geometry>
-            <xacro:material_kuka_orange/>
-        </visual>
-        <collision>
-            <origin xyz="0 0 0" rpy="0 0 0"/>
-            <geometry>
-                <mesh filename="package://${package_name}/meshes/kr10_r1100_sixx/collision/link_4.stl"/>
-            </geometry>
-        </collision>
+      <visual>
+        <origin xyz="0 0 0" rpy="0 0 0"/>
+        <geometry>
+          <mesh filename="package://${package_name}/meshes/kr10_r1100_sixx/visual/link_4.stl"/>
+        </geometry>
+        <xacro:material_kuka_orange/>
+      </visual>
+      <collision>
+        <origin xyz="0 0 0" rpy="0 0 0"/>
+        <geometry>
+          <mesh filename="package://${package_name}/meshes/kr10_r1100_sixx/collision/link_4.stl"/>
+        </geometry>
+      </collision>
     </link>
     <link name="${prefix}link_5">
-        <visual>
-            <origin xyz="0 0 0" rpy="0 0 0"/>
-            <geometry>
-                <mesh filename="package://${package_name}/meshes/kr10_r1100_sixx/visual/link_5.stl"/>
-            </geometry>
-            <xacro:material_kuka_orange/>
-        </visual>
-        <collision>
-            <origin xyz="0 0 0" rpy="0 0 0"/>
-            <geometry>
-                <mesh filename="package://${package_name}/meshes/kr10_r1100_sixx/collision/link_5.stl"/>
-            </geometry>
-        </collision>
+      <visual>
+        <origin xyz="0 0 0" rpy="0 0 0"/>
+        <geometry>
+          <mesh filename="package://${package_name}/meshes/kr10_r1100_sixx/visual/link_5.stl"/>
+        </geometry>
+        <xacro:material_kuka_orange/>
+      </visual>
+      <collision>
+        <origin xyz="0 0 0" rpy="0 0 0"/>
+        <geometry>
+          <mesh filename="package://${package_name}/meshes/kr10_r1100_sixx/collision/link_5.stl"/>
+        </geometry>
+      </collision>
     </link>
     <link name="${prefix}link_6">
-        <visual>
-            <origin xyz="0 0 0" rpy="0 0 0"/>
-            <geometry>
-                <mesh filename="package://${package_name}/meshes/kr10_r1100_sixx/visual/link_6.stl"/>
-            </geometry>
-            <xacro:material_kuka_pedestal/>
-        </visual>
-        <collision>
-            <origin xyz="0 0 0" rpy="0 0 0"/>
-            <geometry>
-                <mesh filename="package://${package_name}/meshes/kr10_r1100_sixx/collision/link_6.stl"/>
-            </geometry>
-        </collision>
+      <visual>
+        <origin xyz="0 0 0" rpy="0 0 0"/>
+        <geometry>
+          <mesh filename="package://${package_name}/meshes/kr10_r1100_sixx/visual/link_6.stl"/>
+        </geometry>
+        <xacro:material_kuka_pedestal/>
+      </visual>
+      <collision>
+        <origin xyz="0 0 0" rpy="0 0 0"/>
+        <geometry>
+          <mesh filename="package://${package_name}/meshes/kr10_r1100_sixx/collision/link_6.stl"/>
+        </geometry>
+      </collision>
     </link>
     <link name="${prefix}tool0"/>
     <joint name="${prefix}base_link-base" type="fixed">
-    <child link="${prefix}base"/>
-    <parent link="${prefix}base_link"/>
+      <child link="${prefix}base"/>
+      <parent link="${prefix}base_link"/>
     </joint>
     <joint name="${prefix}joint_1" type="revolute">
-        <origin xyz="0 0 0.400" rpy="0 0 0"/>
-        <parent link="${prefix}base_link"/>
-        <child link="${prefix}link_1"/>
-        <axis xyz="0 0 -1"/>
-        <limit effort="0" lower="${radians(-170)}" upper="${radians(170)}" velocity="${radians(300)}"/>
+      <origin xyz="0 0 0.400" rpy="0 0 0"/>
+      <parent link="${prefix}base_link"/>
+      <child link="${prefix}link_1"/>
+      <axis xyz="0 0 -1"/>
+      <limit effort="0" lower="${radians(-170)}" upper="${radians(170)}" velocity="${radians(300)}"/>
     </joint>
     <joint name="${prefix}joint_2" type="revolute">
-        <origin xyz="0.025 0 0" rpy="0 0 0"/>
-        <parent link="${prefix}link_1"/>
-        <child link="${prefix}link_2"/>
-        <axis xyz="0 1 0"/>
-        <limit effort="0" lower="${radians(-190)}" upper="${radians(45)}" velocity="${radians(225)}"/>
+      <origin xyz="0.025 0 0" rpy="0 0 0"/>
+      <parent link="${prefix}link_1"/>
+      <child link="${prefix}link_2"/>
+      <axis xyz="0 1 0"/>
+      <limit effort="0" lower="${radians(-190)}" upper="${radians(45)}" velocity="${radians(225)}"/>
     </joint>
     <joint name="${prefix}joint_3" type="revolute">
-        <origin xyz="0.560 0 0" rpy="0 0 0"/>
-        <parent link="${prefix}link_2"/>
-        <child link="${prefix}link_3"/>
-        <axis xyz="0 1 0"/>
-        <limit effort="0" lower="${radians(-120)}" upper="${radians(156)}" velocity="${radians(225)}"/>
+      <origin xyz="0.560 0 0" rpy="0 0 0"/>
+      <parent link="${prefix}link_2"/>
+      <child link="${prefix}link_3"/>
+      <axis xyz="0 1 0"/>
+      <limit effort="0" lower="${radians(-120)}" upper="${radians(156)}" velocity="${radians(225)}"/>
     </joint>
     <joint name="${prefix}joint_4" type="revolute">
-        <origin xyz="0 0 0.035" rpy="0 0 0"/>
-        <parent link="${prefix}link_3"/>
-        <child link="${prefix}link_4"/>
-        <axis xyz="-1 0 0"/>
-        <limit effort="0" lower="${radians(-185)}" upper="${radians(185)}" velocity="${radians(381)}"/>
+      <origin xyz="0 0 0.035" rpy="0 0 0"/>
+      <parent link="${prefix}link_3"/>
+      <child link="${prefix}link_4"/>
+      <axis xyz="-1 0 0"/>
+      <limit effort="0" lower="${radians(-185)}" upper="${radians(185)}" velocity="${radians(381)}"/>
     </joint>
     <joint name="${prefix}joint_5" type="revolute">
-        <origin xyz="0.515 0 0" rpy="0 0 0"/>
-        <parent link="${prefix}link_4"/>
-        <child link="${prefix}link_5"/>
-        <axis xyz="0 1 0"/>
-        <limit effort="0" lower="${radians(-120)}" upper="${radians(120)}" velocity="${radians(311)}"/>
+      <origin xyz="0.515 0 0" rpy="0 0 0"/>
+      <parent link="${prefix}link_4"/>
+      <child link="${prefix}link_5"/>
+      <axis xyz="0 1 0"/>
+      <limit effort="0" lower="${radians(-120)}" upper="${radians(120)}" velocity="${radians(311)}"/>
     </joint>
     <joint name="${prefix}joint_6" type="revolute">
-        <origin xyz="0.080 0 0" rpy="0 0 0"/>
-        <parent link="${prefix}link_5"/>
-        <child link="${prefix}link_6"/>
-        <axis xyz="-1 0 0"/>
-        <limit effort="0" lower="${radians(-350)}" upper="${radians(350)}" velocity="${radians(492)}"/>
+      <origin xyz="0.080 0 0" rpy="0 0 0"/>
+      <parent link="${prefix}link_5"/>
+      <child link="${prefix}link_6"/>
+      <axis xyz="-1 0 0"/>
+      <limit effort="0" lower="${radians(-350)}" upper="${radians(350)}" velocity="${radians(492)}"/>
     </joint>
     <joint name="${prefix}link6-flange" type="fixed">
-        <parent link="${prefix}link_6"/>
-        <child link="${prefix}flange"/>
-        <origin xyz="0 0 0" rpy="0 0 0"/>
+      <parent link="${prefix}link_6"/>
+      <child link="${prefix}flange"/>
+      <origin xyz="0 0 0" rpy="0 0 0"/>
     </joint>
     <joint name="${prefix}link6-tool0" type="fixed">
-        <parent link="${prefix}link_6"/>
-        <child link="${prefix}tool0"/>
-        <origin xyz="0 0 0" rpy="0 ${radians(90)} 0"/>
+      <parent link="${prefix}link_6"/>
+      <child link="${prefix}tool0"/>
+      <origin xyz="0 0 0" rpy="0 ${radians(90)} 0"/>
     </joint>
-</xacro:macro>
+  </xacro:macro>
 </robot>

File: kuka_agilus_support/urdf/kr_agilus_ros2_control_macro.xacro (robot description, xacro)
@@ -12,9 +12,9 @@
     <!-- ros2 control -->
     <ros2_control name="${name}" type="system" is_async="${is_async}" rw_rate="250">
-        <xacro:if value="${is_async}">
-          <properties>
-              <async affinity="${async_affinity}" scheduling_policy="${scheduling_policy}" print_warnings="false" thread_priority="${async_thread_priority}"/>
-          </properties>
-        </xacro:if>
+      <xacro:if value="${is_async}">
+        <properties>
+          <async affinity="${async_affinity}" scheduling_policy="${scheduling_policy}" print_warnings="false" thread_priority="${async_thread_priority}"/>
+        </properties>
+      </xacro:if>
       <hardware>
         <param name="interface_prefix">${prefix}</param>

File: kuka_cybertech_support/urdf/kr_cybertech_ros2_control_macro.xacro (robot description, xacro)
@@ -12,9 +12,9 @@
     <!-- ros2 control -->
     <ros2_control name="${name}" type="system" is_async="${is_async}">
-        <xacro:if value="${is_async}">
-          <properties>
-              <async affinity="${async_affinity}" scheduling_policy="${scheduling_policy}" print_warnings="false" thread_priority="${async_thread_priority}"/>
-          </properties>
-        </xacro:if>
+      <xacro:if value="${is_async}">
+        <properties>
+          <async affinity="${async_affinity}" scheduling_policy="${scheduling_policy}" print_warnings="false" thread_priority="${async_thread_priority}"/>
+        </properties>
+      </xacro:if>
       <hardware>
         <param name="interface_prefix">${prefix}</param>

File: kuka_fortec_support/urdf/kr_fortec_ros2_control_macro.xacro (robot description, xacro)
@@ -14,5 +14,5 @@
       <xacro:if value="${is_async}">
         <properties>
-            <async affinity="${async_affinity}" scheduling_policy="${scheduling_policy}" print_warnings="false" thread_priority="${async_thread_priority}"/>
+          <async affinity="${async_affinity}" scheduling_policy="${scheduling_policy}" print_warnings="false" thread_priority="${async_thread_priority}"/>
         </properties>
       </xacro:if>

File: kuka_iontec_support/urdf/kr_iontec_ros2_control_macro.xacro (robot description, xacro)
@@ -14,5 +14,5 @@
       <xacro:if value="${is_async}">
         <properties>
-            <async affinity="${async_affinity}" scheduling_policy="${scheduling_policy}" print_warnings="false" thread_priority="${async_thread_priority}"/>
+          <async affinity="${async_affinity}" scheduling_policy="${scheduling_policy}" print_warnings="false" thread_priority="${async_thread_priority}"/>
         </properties>
       </xacro:if>

File: kuka_lbr_iico_support/urdf/lbr_iico_ros2_control_macro.xacro (robot description, xacro)
@@ -14,5 +14,5 @@
       <xacro:if value="${is_async}">
         <properties>
-            <async affinity="${async_affinity}" scheduling_policy="${scheduling_policy}" print_warnings="false" thread_priority="${async_thread_priority}"/>
+          <async affinity="${async_affinity}" scheduling_policy="${scheduling_policy}" print_warnings="false" thread_priority="${async_thread_priority}"/>
         </properties>
       </xacro:if>

File: kuka_lbr_iisy_support/urdf/lbr_iisy_ros2_control_macro.xacro (robot description, xacro)
@@ -14,5 +14,5 @@
       <xacro:if value="${is_async}">
         <properties>
-            <async affinity="${async_affinity}" scheduling_policy="${scheduling_policy}" print_warnings="false" thread_priority="${async_thread_priority}"/>
+          <async affinity="${async_affinity}" scheduling_policy="${scheduling_policy}" print_warnings="false" thread_priority="${async_thread_priority}"/>
         </properties>
       </xacro:if>

File: kuka_lbr_iiwa_support/urdf/lbr_iiwa_ros2_control_macro.xacro (robot description, xacro)
@@ -11,5 +11,5 @@
       <xacro:if value="${is_async}">
         <properties>
-            <async affinity="${async_affinity}" scheduling_policy="${scheduling_policy}" print_warnings="false" thread_priority="${async_thread_priority}"/>
+          <async affinity="${async_affinity}" scheduling_policy="${scheduling_policy}" print_warnings="false" thread_priority="${async_thread_priority}"/>
         </properties>
       </xacro:if>

File: kuka_quantec_support/urdf/kr_quantec_ros2_control_macro.xacro (robot description, xacro)
@@ -14,5 +14,5 @@
       <xacro:if value="${is_async}">
         <properties>
-            <async affinity="${async_affinity}" scheduling_policy="${scheduling_policy}" print_warnings="false" thread_priority="${async_thread_priority}"/>
+          <async affinity="${async_affinity}" scheduling_policy="${scheduling_policy}" print_warnings="false" thread_priority="${async_thread_priority}"/>
         </properties>
       </xacro:if>
