Commit message: scheduling policy argument added to new models
Signed-off-by: Sachin Kumar <sachinkum123567@gmail.com>

File: kuka_iontec_support/urdf/kr50_r2500.urdf.xacro (robot description, xacro)
@@ -8,4 +8,5 @@
   <xacro:arg name="mode" default="hardware"/>
   <xacro:arg name="use_gpio" default="false"/>
+  <xacro:arg name="scheduling_policy" default="detached"/>
   <xacro:arg name="roundtrip_time" default="0"/>
   <xacro:arg name="client_ip" default="0.0.0.0"/>
@@ -25,5 +26,5 @@
   <xacro:arg name="yaw" default="0"/>
   <xacro:arg name="rsi_xml_config_file" default=""/>
-  <xacro:kuka_iontec_ros2_control name="$(arg prefix)kr50_r2500" driver_version="$(arg driver_version)" client_ip="$(arg client_ip)" client_port="$(arg client_port)" mxa_client_port="$(arg mxa_client_port)" controller_ip="$(arg controller_ip)" prefix="$(arg prefix)" mode="$(arg mode)" use_gpio="$(arg use_gpio)" roundtrip_time="$(arg roundtrip_time)" verify_robot_model="$(arg verify_robot_model)" rsi_xml_config_file="$(arg rsi_xml_config_file)" is_async="$(arg is_async)" async_thread_priority="$(arg async_thread_priority)" async_affinity="$(arg async_affinity)">
+  <xacro:kuka_iontec_ros2_control name="$(arg prefix)kr50_r2500" driver_version="$(arg driver_version)" client_ip="$(arg client_ip)" client_port="$(arg client_port)" mxa_client_port="$(arg mxa_client_port)" controller_ip="$(arg controller_ip)" prefix="$(arg prefix)" mode="$(arg mode)" use_gpio="$(arg use_gpio)" roundtrip_time="$(arg roundtrip_time)" verify_robot_model="$(arg verify_robot_model)" rsi_xml_config_file="$(arg rsi_xml_config_file)" is_async="$(arg is_async)" scheduling_policy="$(arg scheduling_policy)" async_thread_priority="$(arg async_thread_priority)" async_affinity="$(arg async_affinity)">
     <ext_axes_ros2_control_joints/>
   </xacro:kuka_iontec_ros2_control>

File: kuka_lbr_iico_support/urdf/lbr_iico12_r1260.urdf.xacro (robot description, xacro)
@@ -19,4 +19,5 @@
   <xacro:arg name="mode" default="hardware"/>
   <xacro:arg name="use_gpio" default="false"/>
+  <xacro:arg name="scheduling_policy" default="detached"/>
   <xacro:arg name="roundtrip_time" default="0"/>
   <xacro:arg name="client_ip" default="0.0.0.0"/>
@@ -26,5 +27,5 @@
   <xacro:arg name="verify_robot_model" default="true"/>
   <xacro:arg name="rsi_xml_config_file" default=""/>
-  <xacro:kuka_lbr_iico_ros2_control name="$(arg prefix)lbr_iico12_r1260" driver_version="$(arg driver_version)" client_ip="$(arg client_ip)" client_port="$(arg client_port)" mxa_client_port="$(arg mxa_client_port)" controller_ip="$(arg controller_ip)" prefix="$(arg prefix)" mode="$(arg mode)" use_gpio="$(arg use_gpio)" roundtrip_time="$(arg roundtrip_time)" verify_robot_model="$(arg verify_robot_model)" rsi_xml_config_file="$(arg rsi_xml_config_file)" is_async="$(arg is_async)" async_thread_priority="$(arg async_thread_priority)" async_affinity="$(arg async_affinity)">
+  <xacro:kuka_lbr_iico_ros2_control name="$(arg prefix)lbr_iico12_r1260" driver_version="$(arg driver_version)" client_ip="$(arg client_ip)" client_port="$(arg client_port)" mxa_client_port="$(arg mxa_client_port)" controller_ip="$(arg controller_ip)" prefix="$(arg prefix)" mode="$(arg mode)" use_gpio="$(arg use_gpio)" roundtrip_time="$(arg roundtrip_time)" verify_robot_model="$(arg verify_robot_model)" rsi_xml_config_file="$(arg rsi_xml_config_file)" is_async="$(arg is_async)" scheduling_policy="$(arg scheduling_policy)" async_thread_priority="$(arg async_thread_priority)" async_affinity="$(arg async_affinity)">
     <ext_axes_ros2_control_joints/>
   </xacro:kuka_lbr_iico_ros2_control>

File: kuka_lbr_iico_support/urdf/lbr_iico7_r900.urdf.xacro (robot description, xacro)
@@ -19,4 +19,5 @@
   <xacro:arg name="mode" default="hardware"/>
   <xacro:arg name="use_gpio" default="false"/>
+  <xacro:arg name="scheduling_policy" default="detached"/>
   <xacro:arg name="roundtrip_time" default="0"/>
   <xacro:arg name="client_ip" default="0.0.0.0"/>
@@ -26,5 +27,5 @@
   <xacro:arg name="verify_robot_model" default="true"/>
   <xacro:arg name="rsi_xml_config_file" default=""/>
-  <xacro:kuka_lbr_iico_ros2_control name="$(arg prefix)lbr_iico7_r900" driver_version="$(arg driver_version)" client_ip="$(arg client_ip)" client_port="$(arg client_port)" mxa_client_port="$(arg mxa_client_port)" controller_ip="$(arg controller_ip)" prefix="$(arg prefix)" mode="$(arg mode)" use_gpio="$(arg use_gpio)" roundtrip_time="$(arg roundtrip_time)" verify_robot_model="$(arg verify_robot_model)" rsi_xml_config_file="$(arg rsi_xml_config_file)" is_async="$(arg is_async)" async_thread_priority="$(arg async_thread_priority)" async_affinity="$(arg async_affinity)">
+  <xacro:kuka_lbr_iico_ros2_control name="$(arg prefix)lbr_iico7_r900" driver_version="$(arg driver_version)" client_ip="$(arg client_ip)" client_port="$(arg client_port)" mxa_client_port="$(arg mxa_client_port)" controller_ip="$(arg controller_ip)" prefix="$(arg prefix)" mode="$(arg mode)" use_gpio="$(arg use_gpio)" roundtrip_time="$(arg roundtrip_time)" verify_robot_model="$(arg verify_robot_model)" rsi_xml_config_file="$(arg rsi_xml_config_file)" is_async="$(arg is_async)" scheduling_policy="$(arg scheduling_policy)" async_thread_priority="$(arg async_thread_priority)" async_affinity="$(arg async_affinity)">
     <ext_axes_ros2_control_joints/>
   </xacro:kuka_lbr_iico_ros2_control>

File: kuka_lbr_iico_support/urdf/lbr_iico_ros2_control_macro.xacro (robot description, xacro)
@@ -1,5 +1,5 @@
 <?xml version="1.0" encoding="UTF-8"?>
 <robot xmlns:xacro="http://www.ros.org/wiki/xacro">
-  <xacro:macro name="kuka_lbr_iico_ros2_control" params="name driver_version client_ip client_port mxa_client_port controller_ip prefix mode use_gpio roundtrip_time verify_robot_model rsi_xml_config_file is_async async_thread_priority async_affinity gazebo_controller_config_path:=config/fake_hardware_config_6_axis.yaml **ext_axes_ros2_control_joints">
+  <xacro:macro name="kuka_lbr_iico_ros2_control" params="name driver_version client_ip client_port mxa_client_port controller_ip prefix mode use_gpio roundtrip_time verify_robot_model rsi_xml_config_file is_async async_thread_priority async_affinity gazebo_controller_config_path:=config/fake_hardware_config_6_axis.yaml **ext_axes_ros2_control_joints scheduling_policy:=detached">
     <!-- gazebo -->
     <xacro:if value="${mode == 'gazebo'}">
@@ -8,8 +8,10 @@
     </xacro:if>
     <!-- ros2 control -->
-    <ros2_control name="${name}" type="system" is_async="${is_async}">
-      <properties>
-        <async affinity="${async_affinity}" scheduling_policy="detached" print_warnings="false" thread_priority="${async_thread_priority}"/>
-      </properties>
+    <ros2_control name="${name}" type="system" is_async="${is_async}" rw_rate="250">
+      <xacro:if value="${is_async}">
+        <properties>
+            <async affinity="${async_affinity}" scheduling_policy="${scheduling_policy}" print_warnings="false" thread_priority="${async_thread_priority}"/>
+        </properties>
+      </xacro:if>
       <hardware>
         <param name="interface_prefix">${prefix}</param>

File: kuka_lbr_iisy_support/urdf/lbr_iisy8_r930.urdf.xacro (robot description, xacro)
@@ -19,4 +19,5 @@
   <xacro:arg name="mode" default="hardware"/>
   <xacro:arg name="use_gpio" default="false"/>
+  <xacro:arg name="scheduling_policy" default="detached"/>
   <xacro:arg name="roundtrip_time" default="0"/>
   <xacro:arg name="client_ip" default="0.0.0.0"/>
@@ -27,5 +28,5 @@
   <xacro:arg name="qos_config_file" default=""/>
   <xacro:arg name="rsi_xml_config_file" default=""/>
-  <xacro:kuka_lbr_iisy_ros2_control name="$(arg prefix)lbr_iisy8_r930" driver_version="$(arg driver_version)" client_ip="$(arg client_ip)" client_port="$(arg client_port)" mxa_client_port="$(arg mxa_client_port)" controller_ip="$(arg controller_ip)" prefix="$(arg prefix)" mode="$(arg mode)" use_gpio="$(arg use_gpio)" roundtrip_time="$(arg roundtrip_time)" verify_robot_model="$(arg verify_robot_model)" qos_config_file="$(arg qos_config_file)" rsi_xml_config_file="$(arg rsi_xml_config_file)" is_async="$(arg is_async)" async_thread_priority="$(arg async_thread_priority)" async_affinity="$(arg async_affinity)">
+  <xacro:kuka_lbr_iisy_ros2_control name="$(arg prefix)lbr_iisy8_r930" driver_version="$(arg driver_version)" client_ip="$(arg client_ip)" client_port="$(arg client_port)" mxa_client_port="$(arg mxa_client_port)" controller_ip="$(arg controller_ip)" prefix="$(arg prefix)" mode="$(arg mode)" use_gpio="$(arg use_gpio)" roundtrip_time="$(arg roundtrip_time)" verify_robot_model="$(arg verify_robot_model)" qos_config_file="$(arg qos_config_file)" rsi_xml_config_file="$(arg rsi_xml_config_file)" is_async="$(arg is_async)" scheduling_policy="$(arg scheduling_policy)" async_thread_priority="$(arg async_thread_priority)" async_affinity="$(arg async_affinity)">
     <ext_axes_ros2_control_joints/>
   </xacro:kuka_lbr_iisy_ros2_control>

File: kuka_quantec_support/urdf/kr120_r2700_2.urdf.xacro (robot description, xacro)
@@ -16,4 +16,5 @@
   <xacro:arg name="mode" default="hardware"/>
   <xacro:arg name="use_gpio" default="false"/>
+  <xacro:arg name="scheduling_policy" default="detached"/>
   <xacro:arg name="roundtrip_time" default="0"/>
   <xacro:arg name="client_ip" default="0.0.0.0"/>
@@ -26,5 +27,5 @@
   <xacro:arg name="async_affinity" default="[]"/>
   <xacro:arg name="rsi_xml_config_file" default=""/>
-  <xacro:kuka_quantec_ros2_control name="$(arg prefix)kr120_r2700_2" driver_version="$(arg driver_version)" client_ip="$(arg client_ip)" client_port="$(arg client_port)" mxa_client_port="$(arg mxa_client_port)" controller_ip="$(arg controller_ip)" prefix="$(arg prefix)" mode="$(arg mode)" use_gpio="$(arg use_gpio)" roundtrip_time="$(arg roundtrip_time)" verify_robot_model="$(arg verify_robot_model)" rsi_xml_config_file="$(arg rsi_xml_config_file)" is_async="$(arg is_async)" async_thread_priority="$(arg async_thread_priority)" async_affinity="$(arg async_affinity)">
+  <xacro:kuka_quantec_ros2_control name="$(arg prefix)kr120_r2700_2" driver_version="$(arg driver_version)" client_ip="$(arg client_ip)" client_port="$(arg client_port)" mxa_client_port="$(arg mxa_client_port)" controller_ip="$(arg controller_ip)" prefix="$(arg prefix)" mode="$(arg mode)" use_gpio="$(arg use_gpio)" roundtrip_time="$(arg roundtrip_time)" verify_robot_model="$(arg verify_robot_model)" rsi_xml_config_file="$(arg rsi_xml_config_file)" is_async="$(arg is_async)" scheduling_policy="$(arg scheduling_policy)" async_thread_priority="$(arg async_thread_priority)" async_affinity="$(arg async_affinity)">
     <ext_axes_ros2_control_joints/>
   </xacro:kuka_quantec_ros2_control>

File: kuka_quantec_support/urdf/kr210_r3100_ultra.urdf.xacro (robot description, xacro)
@@ -8,4 +8,5 @@
   <xacro:arg name="mode" default="hardware"/>
   <xacro:arg name="use_gpio" default="false"/>
+  <xacro:arg name="scheduling_policy" default="detached"/>
   <xacro:arg name="roundtrip_time" default="0"/>
   <xacro:arg name="client_ip" default="0.0.0.0"/>
@@ -25,5 +26,5 @@
   <xacro:arg name="yaw" default="0"/>
   <xacro:arg name="rsi_xml_config_file" default=""/>
-  <xacro:kuka_quantec_ros2_control name="$(arg prefix)kr210_r3100_ultra" driver_version="$(arg driver_version)" client_ip="$(arg client_ip)" client_port="$(arg client_port)" mxa_client_port="$(arg mxa_client_port)" controller_ip="$(arg controller_ip)" prefix="$(arg prefix)" mode="$(arg mode)" use_gpio="$(arg use_gpio)" roundtrip_time="$(arg roundtrip_time)" verify_robot_model="$(arg verify_robot_model)" rsi_xml_config_file="$(arg rsi_xml_config_file)" is_async="$(arg is_async)" async_thread_priority="$(arg async_thread_priority)" async_affinity="$(arg async_affinity)">
+  <xacro:kuka_quantec_ros2_control name="$(arg prefix)kr210_r3100_ultra" driver_version="$(arg driver_version)" client_ip="$(arg client_ip)" client_port="$(arg client_port)" mxa_client_port="$(arg mxa_client_port)" controller_ip="$(arg controller_ip)" prefix="$(arg prefix)" mode="$(arg mode)" use_gpio="$(arg use_gpio)" roundtrip_time="$(arg roundtrip_time)" verify_robot_model="$(arg verify_robot_model)" rsi_xml_config_file="$(arg rsi_xml_config_file)" is_async="$(arg is_async)" scheduling_policy="$(arg scheduling_policy)" async_thread_priority="$(arg async_thread_priority)" async_affinity="$(arg async_affinity)">
     <ext_axes_ros2_control_joints/>
   </xacro:kuka_quantec_ros2_control>
