Commit message: Expose gpio_config as a configurable xacro argument
Add a gpio_config argument to every ros2_control macro that supports
use_gpio, defaulting to the existing kuka_rsi_driver gpio_config.xacro
when left empty. This lets a launch file point use_gpio at a custom
GPIO xacro file, for example to describe external IOs, instead of
always including the driver's default config.

Wire the argument through every per-model urdf.xacro so it can be set
from the top level.

Co-Authored-By: Claude Sonnet 5 <noreply@anthropic.com>

File: kuka_cybertech_support/urdf/kr12_r1450_3_hw.urdf.xacro (robot description, xacro)
@@ -8,4 +8,5 @@
   <xacro:arg name="mode" default="hardware"/>
   <xacro:arg name="use_gpio" default="false"/>
+  <xacro:arg name="gpio_config" default=""/>
   <xacro:arg name="scheduling_policy" default="detached"/>
   <xacro:arg name="roundtrip_time" default="0"/>
@@ -26,5 +27,5 @@
   <xacro:arg name="yaw" default="0"/>
   <xacro:arg name="rsi_xml_config_file" default=""/>
-  <xacro:kuka_cybertech_ros2_control name="$(arg prefix)kr12_r1450_3_hw" driver_version="$(arg driver_version)" client_ip="$(arg client_ip)" client_port="$(arg client_port)" mxa_client_port="$(arg mxa_client_port)" controller_ip="$(arg controller_ip)" prefix="$(arg prefix)" mode="$(arg mode)" use_gpio="$(arg use_gpio)" roundtrip_time="$(arg roundtrip_time)" verify_robot_model="$(arg verify_robot_model)" rsi_xml_config_file="$(arg rsi_xml_config_file)" is_async="$(arg is_async)" scheduling_policy="$(arg scheduling_policy)" async_thread_priority="$(arg async_thread_priority)" async_affinity="$(arg async_affinity)">
+  <xacro:kuka_cybertech_ros2_control name="$(arg prefix)kr12_r1450_3_hw" driver_version="$(arg driver_version)" client_ip="$(arg client_ip)" client_port="$(arg client_port)" mxa_client_port="$(arg mxa_client_port)" controller_ip="$(arg controller_ip)" prefix="$(arg prefix)" mode="$(arg mode)" use_gpio="$(arg use_gpio)" gpio_config="$(arg gpio_config)" roundtrip_time="$(arg roundtrip_time)" verify_robot_model="$(arg verify_robot_model)" rsi_xml_config_file="$(arg rsi_xml_config_file)" is_async="$(arg is_async)" scheduling_policy="$(arg scheduling_policy)" async_thread_priority="$(arg async_thread_priority)" async_affinity="$(arg async_affinity)">
     <ext_axes_ros2_control_joints/>
   </xacro:kuka_cybertech_ros2_control>

File: kuka_cybertech_support/urdf/kr16_r1610_2.urdf.xacro (robot description, xacro)
@@ -8,4 +8,5 @@
   <xacro:arg name="mode" default="hardware"/>
   <xacro:arg name="use_gpio" default="false"/>
+  <xacro:arg name="gpio_config" default=""/>
   <xacro:arg name="scheduling_policy" default="detached"/>
   <xacro:arg name="roundtrip_time" default="0"/>
@@ -26,5 +27,5 @@
   <xacro:arg name="yaw" default="0"/>
   <xacro:arg name="rsi_xml_config_file" default=""/>
-  <xacro:kuka_cybertech_ros2_control name="$(arg prefix)kr16_r1610_2" driver_version="$(arg driver_version)" client_ip="$(arg client_ip)" client_port="$(arg client_port)" mxa_client_port="$(arg mxa_client_port)" controller_ip="$(arg controller_ip)" prefix="$(arg prefix)" mode="$(arg mode)" use_gpio="$(arg use_gpio)" roundtrip_time="$(arg roundtrip_time)" verify_robot_model="$(arg verify_robot_model)" rsi_xml_config_file="$(arg rsi_xml_config_file)" is_async="$(arg is_async)" scheduling_policy="$(arg scheduling_policy)" async_thread_priority="$(arg async_thread_priority)" async_affinity="$(arg async_affinity)">
+  <xacro:kuka_cybertech_ros2_control name="$(arg prefix)kr16_r1610_2" driver_version="$(arg driver_version)" client_ip="$(arg client_ip)" client_port="$(arg client_port)" mxa_client_port="$(arg mxa_client_port)" controller_ip="$(arg controller_ip)" prefix="$(arg prefix)" mode="$(arg mode)" use_gpio="$(arg use_gpio)" gpio_config="$(arg gpio_config)" roundtrip_time="$(arg roundtrip_time)" verify_robot_model="$(arg verify_robot_model)" rsi_xml_config_file="$(arg rsi_xml_config_file)" is_async="$(arg is_async)" scheduling_policy="$(arg scheduling_policy)" async_thread_priority="$(arg async_thread_priority)" async_affinity="$(arg async_affinity)">
     <ext_axes_ros2_control_joints/>
   </xacro:kuka_cybertech_ros2_control>

File: kuka_cybertech_support/urdf/kr16_r2010_2.urdf.xacro (robot description, xacro)
@@ -8,4 +8,5 @@
   <xacro:arg name="mode" default="hardware"/>
   <xacro:arg name="use_gpio" default="false"/>
+  <xacro:arg name="gpio_config" default=""/>
   <xacro:arg name="scheduling_policy" default="detached"/>
   <xacro:arg name="roundtrip_time" default="0"/>
@@ -26,5 +27,5 @@
   <xacro:arg name="yaw" default="0"/>
   <xacro:arg name="rsi_xml_config_file" default=""/>
-  <xacro:kuka_cybertech_ros2_control name="$(arg prefix)kr16_r2010_2" driver_version="$(arg driver_version)" client_ip="$(arg client_ip)" client_port="$(arg client_port)" mxa_client_port="$(arg mxa_client_port)" controller_ip="$(arg controller_ip)" prefix="$(arg prefix)" mode="$(arg mode)" use_gpio="$(arg use_gpio)" roundtrip_time="$(arg roundtrip_time)" verify_robot_model="$(arg verify_robot_model)" rsi_xml_config_file="$(arg rsi_xml_config_file)" is_async="$(arg is_async)" scheduling_policy="$(arg scheduling_policy)" async_thread_priority="$(arg async_thread_priority)" async_affinity="$(arg async_affinity)">
+  <xacro:kuka_cybertech_ros2_control name="$(arg prefix)kr16_r2010_2" driver_version="$(arg driver_version)" client_ip="$(arg client_ip)" client_port="$(arg client_port)" mxa_client_port="$(arg mxa_client_port)" controller_ip="$(arg controller_ip)" prefix="$(arg prefix)" mode="$(arg mode)" use_gpio="$(arg use_gpio)" gpio_config="$(arg gpio_config)" roundtrip_time="$(arg roundtrip_time)" verify_robot_model="$(arg verify_robot_model)" rsi_xml_config_file="$(arg rsi_xml_config_file)" is_async="$(arg is_async)" scheduling_policy="$(arg scheduling_policy)" async_thread_priority="$(arg async_thread_priority)" async_affinity="$(arg async_affinity)">
     <ext_axes_ros2_control_joints/>
   </xacro:kuka_cybertech_ros2_control>

File: kuka_cybertech_support/urdf/kr20_r1810_2.urdf.xacro (robot description, xacro)
@@ -8,4 +8,5 @@
   <xacro:arg name="mode" default="hardware"/>
   <xacro:arg name="use_gpio" default="false"/>
+  <xacro:arg name="gpio_config" default=""/>
   <xacro:arg name="scheduling_policy" default="detached"/>
   <xacro:arg name="roundtrip_time" default="0"/>
@@ -26,5 +27,5 @@
   <xacro:arg name="yaw" default="0"/>
   <xacro:arg name="rsi_xml_config_file" default=""/>
-  <xacro:kuka_cybertech_ros2_control name="$(arg prefix)kr20_r1810_2" driver_version="$(arg driver_version)" client_ip="$(arg client_ip)" client_port="$(arg client_port)" mxa_client_port="$(arg mxa_client_port)" controller_ip="$(arg controller_ip)" prefix="$(arg prefix)" mode="$(arg mode)" use_gpio="$(arg use_gpio)" roundtrip_time="$(arg roundtrip_time)" verify_robot_model="$(arg verify_robot_model)" rsi_xml_config_file="$(arg rsi_xml_config_file)" is_async="$(arg is_async)" scheduling_policy="$(arg scheduling_policy)" async_thread_priority="$(arg async_thread_priority)" async_affinity="$(arg async_affinity)">
+  <xacro:kuka_cybertech_ros2_control name="$(arg prefix)kr20_r1810_2" driver_version="$(arg driver_version)" client_ip="$(arg client_ip)" client_port="$(arg client_port)" mxa_client_port="$(arg mxa_client_port)" controller_ip="$(arg controller_ip)" prefix="$(arg prefix)" mode="$(arg mode)" use_gpio="$(arg use_gpio)" gpio_config="$(arg gpio_config)" roundtrip_time="$(arg roundtrip_time)" verify_robot_model="$(arg verify_robot_model)" rsi_xml_config_file="$(arg rsi_xml_config_file)" is_async="$(arg is_async)" scheduling_policy="$(arg scheduling_policy)" async_thread_priority="$(arg async_thread_priority)" async_affinity="$(arg async_affinity)">
     <ext_axes_ros2_control_joints/>
   </xacro:kuka_cybertech_ros2_control>

File: kuka_cybertech_support/urdf/kr20_r1820_2_e.urdf.xacro (robot description, xacro)
@@ -20,4 +20,5 @@
   <xacro:arg name="mode" default="hardware"/>
   <xacro:arg name="use_gpio" default="false"/>
+  <xacro:arg name="gpio_config" default=""/>
   <xacro:arg name="scheduling_policy" default="detached"/>
   <xacro:arg name="roundtrip_time" default="0"/>
@@ -27,5 +28,5 @@
   <xacro:arg name="controller_ip" default="0.0.0.0"/>
   <xacro:arg name="verify_robot_model" default="true"/>
-  <xacro:kuka_cybertech_ros2_control name="$(arg prefix)kr20_r1820_2_e" driver_version="$(arg driver_version)" client_ip="$(arg client_ip)" client_port="$(arg client_port)" mxa_client_port="$(arg mxa_client_port)" controller_ip="$(arg controller_ip)" prefix="$(arg prefix)" mode="$(arg mode)" use_gpio="$(arg use_gpio)" roundtrip_time="$(arg roundtrip_time)" verify_robot_model="$(arg verify_robot_model)" rsi_xml_config_file="$(arg rsi_xml_config_file)" is_async="$(arg is_async)" scheduling_policy="$(arg scheduling_policy)" async_thread_priority="$(arg async_thread_priority)" async_affinity="$(arg async_affinity)">
+  <xacro:kuka_cybertech_ros2_control name="$(arg prefix)kr20_r1820_2_e" driver_version="$(arg driver_version)" client_ip="$(arg client_ip)" client_port="$(arg client_port)" mxa_client_port="$(arg mxa_client_port)" controller_ip="$(arg controller_ip)" prefix="$(arg prefix)" mode="$(arg mode)" use_gpio="$(arg use_gpio)" gpio_config="$(arg gpio_config)" roundtrip_time="$(arg roundtrip_time)" verify_robot_model="$(arg verify_robot_model)" rsi_xml_config_file="$(arg rsi_xml_config_file)" is_async="$(arg is_async)" scheduling_policy="$(arg scheduling_policy)" async_thread_priority="$(arg async_thread_priority)" async_affinity="$(arg async_affinity)">
     <ext_axes_ros2_control_joints/>
   </xacro:kuka_cybertech_ros2_control>

File: kuka_cybertech_support/urdf/kr35_r1840_3.urdf.xacro (robot description, xacro)
@@ -19,4 +19,5 @@
   <xacro:arg name="mode" default="hardware"/>
   <xacro:arg name="use_gpio" default="false"/>
+  <xacro:arg name="gpio_config" default=""/>
   <xacro:arg name="scheduling_policy" default="detached"/>
   <xacro:arg name="roundtrip_time" default="0"/>
@@ -27,5 +28,5 @@
   <xacro:arg name="verify_robot_model" default="true"/>
   <xacro:arg name="rsi_xml_config_file" default=""/>
-  <xacro:kuka_cybertech_ros2_control name="$(arg prefix)kr35_r1840_3" driver_version="$(arg driver_version)" client_ip="$(arg client_ip)" client_port="$(arg client_port)" mxa_client_port="$(arg mxa_client_port)" controller_ip="$(arg controller_ip)" prefix="$(arg prefix)" mode="$(arg mode)" use_gpio="$(arg use_gpio)" roundtrip_time="$(arg roundtrip_time)" verify_robot_model="$(arg verify_robot_model)" rsi_xml_config_file="$(arg rsi_xml_config_file)" is_async="$(arg is_async)" scheduling_policy="$(arg scheduling_policy)" async_thread_priority="$(arg async_thread_priority)" async_affinity="$(arg async_affinity)">
+  <xacro:kuka_cybertech_ros2_control name="$(arg prefix)kr35_r1840_3" driver_version="$(arg driver_version)" client_ip="$(arg client_ip)" client_port="$(arg client_port)" mxa_client_port="$(arg mxa_client_port)" controller_ip="$(arg controller_ip)" prefix="$(arg prefix)" mode="$(arg mode)" use_gpio="$(arg use_gpio)" gpio_config="$(arg gpio_config)" roundtrip_time="$(arg roundtrip_time)" verify_robot_model="$(arg verify_robot_model)" rsi_xml_config_file="$(arg rsi_xml_config_file)" is_async="$(arg is_async)" scheduling_policy="$(arg scheduling_policy)" async_thread_priority="$(arg async_thread_priority)" async_affinity="$(arg async_affinity)">
     <ext_axes_ros2_control_joints/>
   </xacro:kuka_cybertech_ros2_control>

File: kuka_cybertech_support/urdf/kr35_r1840_3_hw.urdf.xacro (robot description, xacro)
@@ -19,4 +19,5 @@
   <xacro:arg name="mode" default="hardware"/>
   <xacro:arg name="use_gpio" default="false"/>
+  <xacro:arg name="gpio_config" default=""/>
   <xacro:arg name="roundtrip_time" default="0"/>
   <xacro:arg name="client_ip" default="0.0.0.0"/>
@@ -26,5 +27,5 @@
   <xacro:arg name="verify_robot_model" default="true"/>
   <xacro:arg name="rsi_xml_config_file" default=""/>
-  <xacro:kuka_cybertech_ros2_control name="$(arg prefix)kr35_r1840_3_hw" driver_version="$(arg driver_version)" client_ip="$(arg client_ip)" client_port="$(arg client_port)" mxa_client_port="$(arg mxa_client_port)" controller_ip="$(arg controller_ip)" prefix="$(arg prefix)" mode="$(arg mode)" use_gpio="$(arg use_gpio)" roundtrip_time="$(arg roundtrip_time)" verify_robot_model="$(arg verify_robot_model)" rsi_xml_config_file="$(arg rsi_xml_config_file)" is_async="$(arg is_async)" async_thread_priority="$(arg async_thread_priority)" async_affinity="$(arg async_affinity)">
+  <xacro:kuka_cybertech_ros2_control name="$(arg prefix)kr35_r1840_3_hw" driver_version="$(arg driver_version)" client_ip="$(arg client_ip)" client_port="$(arg client_port)" mxa_client_port="$(arg mxa_client_port)" controller_ip="$(arg controller_ip)" prefix="$(arg prefix)" mode="$(arg mode)" use_gpio="$(arg use_gpio)" gpio_config="$(arg gpio_config)" roundtrip_time="$(arg roundtrip_time)" verify_robot_model="$(arg verify_robot_model)" rsi_xml_config_file="$(arg rsi_xml_config_file)" is_async="$(arg is_async)" async_thread_priority="$(arg async_thread_priority)" async_affinity="$(arg async_affinity)">
     <ext_axes_ros2_control_joints/>
   </xacro:kuka_cybertech_ros2_control>

File: kuka_cybertech_support/urdf/kr8_r1440_2_arc_hw.urdf.xacro (robot description, xacro)
@@ -8,4 +8,5 @@
   <xacro:arg name="mode" default="hardware"/>
   <xacro:arg name="use_gpio" default="false"/>
+  <xacro:arg name="gpio_config" default=""/>
   <xacro:arg name="scheduling_policy" default="detached"/>
   <xacro:arg name="roundtrip_time" default="0"/>
@@ -26,5 +27,5 @@
   <xacro:arg name="yaw" default="0"/>
   <xacro:arg name="rsi_xml_config_file" default=""/>
-  <xacro:kuka_cybertech_ros2_control name="$(arg prefix)kr8_r1440_2_arc_hw" driver_version="$(arg driver_version)" client_ip="$(arg client_ip)" client_port="$(arg client_port)" mxa_client_port="$(arg mxa_client_port)" controller_ip="$(arg controller_ip)" prefix="$(arg prefix)" mode="$(arg mode)" use_gpio="$(arg use_gpio)" roundtrip_time="$(arg roundtrip_time)" verify_robot_model="$(arg verify_robot_model)" rsi_xml_config_file="$(arg rsi_xml_config_file)" is_async="$(arg is_async)" scheduling_policy="$(arg scheduling_policy)" async_thread_priority="$(arg async_thread_priority)" async_affinity="$(arg async_affinity)">
+  <xacro:kuka_cybertech_ros2_control name="$(arg prefix)kr8_r1440_2_arc_hw" driver_version="$(arg driver_version)" client_ip="$(arg client_ip)" client_port="$(arg client_port)" mxa_client_port="$(arg mxa_client_port)" controller_ip="$(arg controller_ip)" prefix="$(arg prefix)" mode="$(arg mode)" use_gpio="$(arg use_gpio)" gpio_config="$(arg gpio_config)" roundtrip_time="$(arg roundtrip_time)" verify_robot_model="$(arg verify_robot_model)" rsi_xml_config_file="$(arg rsi_xml_config_file)" is_async="$(arg is_async)" scheduling_policy="$(arg scheduling_policy)" async_thread_priority="$(arg async_thread_priority)" async_affinity="$(arg async_affinity)">
     <ext_axes_ros2_control_joints/>
   </xacro:kuka_cybertech_ros2_control>
